File: AlternativeDrivers.sch (KiCad schematic (older format))
At the start: 72 parts, among them Q1 BUK7M12-40EX, Q2 BUK7M12-40EX, Q3 BUK7M12-40EX, Q4 BUK7M12-40EX, U12 VNH5019A-E, U13 VNH5019A-E, U14 VNH5019A-E, U15 VNH5019A-E

Commit message: Rev B
Parts:
- C14, C15, C17, C19, C22, C23, C25, C27: DigiKey (none) -> 399-1100-1-ND
- C16, C18, C24, C26: DigiKey (none) -> 399-10532-1-ND
- D10, D11, D12, D9: DigiKey (none) -> 1497-1383-1-ND
- Q1, Q2, Q3, Q4: DigiKey (none) -> 1727-2556-1-ND
- R11, R12, R13, R14, R15, R16, R26, R27, R30, R31, R32, R33, R36, R37, R38, R39, R40, R41, R48, R49, R52, R53, R54, R55: DigiKey (none) -> 311-1.0KGRCT-ND
- R17, R18, R28, R29, R42, R43, R50, R51: DigiKey (none) -> 311-10KGRCT-ND
- R22, R23, R24, R25, R34, R35, R44, R45, R46, R47, R56, R57: DigiKey (none) -> RR08P4.7KDCT-ND
- U12, U13, U14, U15: DigiKey (none) -> 497-13073-1-ND
