File: Motors.sch (KiCad schematic (older format))
At the start: 14 parts, among them J2 LEFT_MOTOR, J3 RIGHT_MOTOR, U3 VNH5019, U4 VNH5019

Commit message: Added BOM
Parts:
- R11, R13, R15, R17: DigiKey (none) -> RMCF0201FT270RCT-ND
- R12, R14, R16, R18: DigiKey (none) -> RR08P560DCT-ND
Changed lines of the file:
@@
 F 2 "Resistor_SMD:R_0603_1608Metric_Pad1.05x0.95mm_HandSolder" H 3300 1650 50  0001 C CNN
 F 3 "~" H 3300 1650 50  0001 C CNN
+F 4 " RMCF0201FT270RCT-ND " H 3300 1650 50  0001 C CNN "DigiKey"
 	1    3300 1650
 	1    0    0    -1
@@
 F 2 "Resistor_SMD:R_0603_1608Metric_Pad1.05x0.95mm_HandSolder" H 3300 2050 50  0001 C CNN
 F 3 "~" H 3300 2050 50  0001 C CNN
+F 4 " RR08P560DCT-ND " H 3300 2050 50  0001 C CNN "DigiKey"
 	1    3300 2050
 	1    0    0    -1
@@
 F 2 "Resistor_SMD:R_0603_1608Metric_Pad1.05x0.95mm_HandSolder" H 3300 2450 50  0001 C CNN
 F 3 "~" H 3300 2450 50  0001 C CNN
+F 4 " RMCF0201FT270RCT-ND " H 3300 2450 50  0001 C CNN "DigiKey"
 	1    3300 2450
 	1    0    0    -1
@@
 F 2 "Resistor_SMD:R_0603_1608Metric_Pad1.05x0.95mm_HandSolder" H 3300 2850 50  0001 C CNN
 F 3 "~" H 3300 2850 50  0001 C CNN
+F 4 " RR08P560DCT-ND " H 3300 2850 50  0001 C CNN "DigiKey"
 	1    3300 2850
 	1    0    0    -1
@@
 F 2 "Resistor_SMD:R_0603_1608Metric_Pad1.05x0.95mm_HandSolder" H 3300 3300 50  0001 C CNN
 F 3 "~" H 3300 3300 50  0001 C CNN
+F 4 " RMCF0201FT270RCT-ND " H 3300 3300 50  0001 C CNN "DigiKey"
 	1    3300 3300
 	1    0    0    -1
@@
 F 2 "Resistor_SMD:R_0603_1608Metric_Pad1.05x0.95mm_HandSolder" H 3300 3700 50  0001 C CNN
 F 3 "~" H 3300 3700 50  0001 C CNN
+F 4 " RR08P560DCT-ND " H 3300 3700 50  0001 C CNN "DigiKey"
 	1    3300 3700
 	1    0    0    -1
@@
 F 2 "Resistor_SMD:R_0603_1608Metric_Pad1.05x0.95mm_HandSolder" H 3300 4100 50  0001 C CNN
 F 3 "~" H 3300 4100 50  0001 C CNN
+F 4 " RMCF0201FT270RCT-ND " H 3300 4100 50  0001 C CNN "DigiKey"
 	1    3300 4100
 	1    0    0    -1
@@
 F 2 "Resistor_SMD:R_0603_1608Metric_Pad1.05x0.95mm_HandSolder" H 3300 4500 50  0001 C CNN
 F 3 "~" H 3300 4500 50  0001 C CNN
+F 4 " RR08P560DCT-ND " H 3300 4500 50  0001 C CNN "DigiKey"
 	1    3300 4500
 	1    0    0    -1

Commit message: Some fixes
Parts:
- removed R11, R13, R15, R17: 270Ohm, Resistor_SMD:R_0603_1608Metric_Pad1.05x0.95mm_HandSolder, symbol Device:R_Small
- removed R12, R14, R16, R18: 560Ohm, Resistor_SMD:R_0603_1608Metric_Pad1.05x0.95mm_HandSolder, symbol Device:R_Small
- added C? (x2): 0.1uF, symbol Device:C_Small
- added J? (x2): Screw_Terminal_01x02, symbol Connector:Screw_Terminal_01x02
- added JP? (x2): Jumper_3_Bridged12, symbol Jumper:Jumper_3_Bridged12
- added JP? (x4): Jumper_2_Open, symbol Jumper:Jumper_2_Open
- added U?: TXB0104D, Package_SO:SOIC-14_3.9x8.7mm_P1.27mm, symbol Logic_LevelTranslator:TXB0104D
Connections:
- net +3V3: now also C?.1, JP?.3 (B), JP?.3 (B), U?.1 (VCCA), U?.8 (OE)
- net +5V: now also C?.2, JP?.1 (A), JP?.1 (A), U?.14 (VCCB); no longer J2.4 (ENCODER_VCC), J3.4 (ENCODER_VCC)
- net GND: now also C?.1, C?.2, U?.7 (GND)
- net LEFT_ENCODER_A_3.3V: now also JP?.1 (A), U?.2 (A1)
- net LEFT_ENCODER_A_5V: now also JP?.2 (B), U?.13 (B1)
- net LEFT_ENCODER_B_3.3V: now also JP?.1 (A), U?.3 (A2)
- net LEFT_ENCODER_B_5V: now also JP?.2 (B), U?.12 (B2)
- net LEFT_MOTOR_A: now also J?.2 (Pin_2)
- net LEFT_MOTOR_B: now also J?.1 (Pin_1)
- net RIGHT_ENCODER_A_3.3V: now also JP?.1 (A), U?.4 (A3)
- net RIGHT_ENCODER_A_5V: now also JP?.2 (B), U?.11 (B3)
- net RIGHT_ENCODER_B_3.3V: now also JP?.1 (A), U?.5 (A4)
- net RIGHT_ENCODER_B_5V: now also JP?.2 (B), U?.10 (B4)
- net RIGHT_MOTOR_A: now also J?.2 (Pin_2)
- net RIGHT_MOTOR_B: now also J?.1 (Pin_1)
- net LEFT_MOTOR_INA: now reaches U3.1 (INA)
- net LEFT_MOTOR_INB: now reaches U3.6 (INB)
- net RIGHT_MOTOR_INA: now reaches U4.1 (INA)
- net RIGHT_MOTOR_INB: now reaches U4.6 (INB)
- net LEFT_MOTOR_DIAGA: no longer names the net of U3.2 (ENA/DIAGA)
- net LEFT_MOTOR_DIAGB: no longer names the net of U3.5 (ENB/DIAGB)
- net RIGHT_MOTOR_DIAGA: no longer names the net of U4.2 (ENA/DIAGA)
- net RIGHT_MOTOR_DIAGB: no longer names the net of U4.5 (ENB/DIAGB)
- new net: J2.4 (ENCODER_VCC), JP?.2 (C)
- new net: J3.4 (ENCODER_VCC), JP?.2 (C)
Other:
- moved on the sheet: F2, F3, J2, J3, U3, U4

Commit message: Most of rev B
Parts:
- removed F2, F3: Fuse, Fuse:Fuse_0805_2012Metric_Pad1.15x1.40mm_HandSolder, symbol Device:Fuse
- removed J? (x2): Screw_Terminal_01x02, symbol Connector:Screw_Terminal_01x02
- removed JP? (x4): Jumper_2_Open, symbol Jumper:Jumper_2_Open
- added C10, C11: 0.1uF, Capacitor_SMD:C_0603_1608Metric_Pad1.05x0.95mm_HandSolder, symbol Device:C_Small
- added J10, J11, J12, J9: Screw_Terminal_01x02, TerminalBlock_Phoenix:TerminalBlock_Phoenix_MKDS-3-2-5.08_1x02_P5.08mm_Horizontal, symbol Connector:Screw_Terminal_01x02
- added J7: MOTOR_3, Connector_PinHeader_2.54mm:PinHeader_1x06_P2.54mm_Vertical, symbol pololu_parts:MOTOR_CONNECTOR
- added J8: MOTOR_4, Connector_PinHeader_2.54mm:PinHeader_1x06_P2.54mm_Vertical, symbol pololu_parts:MOTOR_CONNECTOR
- added JP7, JP9: Jumper_3_Bridged12, Jumper:SolderJumper-3_P1.3mm_Bridged12_RoundedPad1.0x1.5mm, symbol Jumper:Jumper_3_Bridged12
- added U10: TXB0104D, Package_SO:SOIC-14_3.9x8.7mm_P1.27mm, symbol Logic_LevelTranslator:TXB0104D
- added U11, U9: VNH5019, TurtlebotController:Pololu_VNH5019_Carrier, symbol pololu_parts:VNH5019
- C8, C9: renamed from C?; footprint (none) -> Capacitor_SMD:C_0603_1608Metric_Pad1.05x0.95mm_HandSolder
- J2: value LEFT_MOTOR -> MOTOR_1
- J3: value RIGHT_MOTOR -> MOTOR_2
- JP6, JP8: renamed from JP?; footprint (none) -> Jumper:SolderJumper-3_P1.3mm_Bridged12_RoundedPad1.0x1.5mm
- gave numbers to parts that had none: 1
Connections:
- net +12V: now also U3.14 (VIN), U4.14 (VIN), U11.14 (VIN), U9.14 (VIN)
- net +3V3: now also C10.1, JP7.3 (B), JP9.3 (B), U10.1 (VCCA), U10.8 (OE), U11.7 (VDD), U9.7 (VDD)
- net +5V: now also C11.2, JP7.1 (A), JP9.1 (A), U10.14 (VCCB)
- net GND: now also C10.2, C11.1, J7.3 (ENCODER_GND), J8.3 (ENCODER_GND), U10.7 (GND), U11.10 (GND), U11.13 (GND), U11.8 (GND), U9.10 (GND), U9.13 (GND), U9.8 (GND)
- net MOTOR_1_DIAGA: now reaches U3.2 (ENA/DIAGA)
- net MOTOR_1_DIAGB: now reaches U3.5 (ENB/DIAGB)
- net MOTOR_2_DIAGA: now reaches U4.2 (ENA/DIAGA)
- net MOTOR_2_DIAGB: now reaches U4.5 (ENB/DIAGB)
- net LEFT_ENCODER_A_3.3V renamed MOTOR_1_ENCODER_A
- net LEFT_ENCODER_A_5V renamed MOTOR_1_ENCODER_A_5V
- net LEFT_ENCODER_B_3.3V renamed MOTOR_1_ENCODER_B
- net LEFT_ENCODER_B_5V renamed MOTOR_1_ENCODER_B_5V
- net LEFT_MOTOR_A renamed MOTOR_1_A
- net MOTOR_1_A: now also J9.2 (Pin_2)
- net LEFT_MOTOR_B renamed MOTOR_1_B
- net MOTOR_1_B: now also J9.1 (Pin_1)
- net LEFT_MOTOR_CURRENT renamed MOTOR_1_CS
- net LEFT_MOTOR_INA renamed MOTOR_1_INA
- net LEFT_MOTOR_INB renamed MOTOR_1_INB
- net LEFT_MOTOR_OUT renamed MOTOR_1_OUT
- net LEFT_MOTOR_PWM renamed MOTOR_1_PWM
- net RIGHT_ENCODER_A_3.3V renamed MOTOR_2_ENCODER_A
- net RIGHT_ENCODER_A_5V renamed MOTOR_2_ENCODER_A_5V
- net RIGHT_ENCODER_B_3.3V renamed MOTOR_2_ENCODER_B
- net RIGHT_ENCODER_B_5V renamed MOTOR_2_ENCODER_B_5V
- net RIGHT_MOTOR_A renamed MOTOR_2_A
- net MOTOR_2_A: now also J10.2 (Pin_2)
- net RIGHT_MOTOR_B renamed MOTOR_2_B
- net MOTOR_2_B: now also J10.1 (Pin_1)
- net RIGHT_MOTOR_CURRENT renamed MOTOR_2_CS
- net RIGHT_MOTOR_INA renamed MOTOR_2_INA
- net RIGHT_MOTOR_INB renamed MOTOR_2_INB
- net RIGHT_MOTOR_OUT renamed MOTOR_2_OUT
- net RIGHT_MOTOR_PWM renamed MOTOR_2_PWM
- new net: J7.4 (ENCODER_VCC), JP7.2 (C)
- new net: J8.4 (ENCODER_VCC), JP9.2 (C)
- new net MOTOR_3_A: J11.2 (Pin_2), J7.1 (MOTOR_RED), U9.11 (OUTA)
- new net MOTOR_3_B: J11.1 (Pin_1), J7.2 (MOTOR_BLACK), U9.12 (OUTB)
- new net MOTOR_3_CS: U9.4 (CS)
- new net MOTOR_3_DIAGA: U9.2 (ENA/DIAGA)
- new net MOTOR_3_DIAGB: U9.5 (ENB/DIAGB)
- new net MOTOR_3_ENCODER_A: U10.2 (A1)
- new net MOTOR_3_ENCODER_A_5V: J7.5 (ENCODER_A), U10.13 (B1)
- new net MOTOR_3_ENCODER_B: U10.3 (A2)
- new net MOTOR_3_ENCODER_B_5V: J7.6 (ENCODER_B), U10.12 (B2)
- new net MOTOR_3_INA: U9.1 (INA)
- new net MOTOR_3_INB: U9.6 (INB)
- new net MOTOR_3_OUT: U9.9 (VOUT)
- new net MOTOR_3_PWM: U9.3 (PWM)
- new net MOTOR_4_A: J12.2 (Pin_2), J8.1 (MOTOR_RED), U11.11 (OUTA)
- new net MOTOR_4_B: J12.1 (Pin_1), J8.2 (MOTOR_BLACK), U11.12 (OUTB)
- new net MOTOR_4_CS: U11.4 (CS)
- new net MOTOR_4_DIAGA: U11.2 (ENA/DIAGA)
- new net MOTOR_4_DIAGB: U11.5 (ENB/DIAGB)
- new net MOTOR_4_ENCODER_A: U10.4 (A3)
- new net MOTOR_4_ENCODER_A_5V: J8.5 (ENCODER_A), U10.11 (B3)
- new net MOTOR_4_ENCODER_B: U10.5 (A4)
- new net MOTOR_4_ENCODER_B_5V: J8.6 (ENCODER_B), U10.10 (B4)
- new net MOTOR_4_INA: U11.1 (INA)
- new net MOTOR_4_INB: U11.6 (INB)
- new net MOTOR_4_OUT: U11.9 (VOUT)
- new net MOTOR_4_PWM: U11.3 (PWM)
Other:
- moved on the sheet: C8, C9, J2, J3, JP6, JP8, U3, U4, U8

Commit message: RevB
Parts:
- added JP14: Jumper_3_Bridged12, Jumper:SolderJumper-3_P1.3mm_Bridged12_RoundedPad1.0x1.5mm, symbol Jumper:Jumper_3_Bridged12
Connections:
- net +3V3: now also JP14.3 (B)
- net +5V: now also JP14.1 (A); no longer C11.2, C9.2, U10.14 (VCCB), U8.14 (VCCB)
- new net: C11.2, C9.2, JP14.2 (C), U10.14 (VCCB), U8.14 (VCCB)
- no-connect marks 0 -> 1
Changed lines of the file:
@@
 	1    0    0    -1
 $EndComp
-$Comp
-L power:+5V #PWR0146
-U 1 1 5EC0369F
-P 2200 5250
-F 0 "#PWR0146" H 2200 5100 50  0001 C CNN
-F 1 "+5V" H 2215 5423 50  0000 C CNN
-F 2 "" H 2200 5250 50  0001 C CNN
-F 3 "" H 2200 5250 50  0001 C CNN
-	1    2200 5250
-	1    0    0    -1
-$EndComp
-Wire Wire Line
-	2200 5250 2200 5650
 Wire Wire Line
 	2200 5650 2200 5800
@@
 	1    0    0    -1
 $EndComp
-$Comp
-L power:+5V #PWR0196
-U 1 1 5EFA5CB7
-P 5150 5250
-F 0 "#PWR0196" H 5150 5100 50  0001 C CNN
-F 1 "+5V" H 5165 5423 50  0000 C CNN
-F 2 "" H 5150 5250 50  0001 C CNN
-F 3 "" H 5150 5250 50  0001 C CNN
-	1    5150 5250
-	1    0    0    -1
-$EndComp
-Wire Wire Line
-	5150 5250 5150 5650
 Wire Wire Line
 	5150 5650 5150 5800
@@
 Wire Wire Line
 	9800 3600 10250 3600
+Wire Wire Line
+	3950 5150 3850 5150
+$Comp
+L power:+3.3V #PWR?
+U 1 1 5EC1A386
+P 3950 5150
+AR Path="/5EC1A386" Ref="#PWR?"  Part="1"
+AR Path="/5E0C61A9/5EC1A386" Ref="#PWR0146"  Part="1"
+F 0 "#PWR0146" H 3950 5000 50  0001 C CNN
+F 1 "+3.3V" V 3965 5278 50  0000 L CNN
+F 2 "" H 3950 5150 50  0001 C CNN
+F 3 "" H 3950 5150 50  0001 C CNN
+	1    3950 5150
+	0    1    1    0
+$EndComp
+$Comp
+L Jumper:Jumper_3_Bridged12 JP14
+U 1 1 5EC1A390
+P 3600 5150
+F 0 "JP14" H 3600 5354 50  0000 C CNN
+F 1 "Jumper_3_Bridged12" H 3600 5263 50  0000 C CNN
+F 2 "Jumper:SolderJumper-3_P1.3mm_Bridged12_RoundedPad1.0x1.5mm" H 3600 5150 50  0001 C CNN
+F 3 "~" H 3600 5150 50  0001 C CNN
+	1    3600 5150
+	1    0    0    -1
+$EndComp
+$Comp
+L power:+5V #PWR?
+U 1 1 5EC1A39A
+P 3350 5150
+AR Path="/5EC1A39A" Ref="#PWR?"  Part="1"
+AR Path="/5E0C61A9/5EC1A39A" Ref="#PWR0196"  Part="1"
+F 0 "#PWR0196" H 3350 5000 50  0001 C CNN
+F 1 "+5V" V 3365 5278 50  0000 L CNN
+F 2 "" H 3350 5150 50  0001 C CNN
+F 3 "" H 3350 5150 50  0001 C CNN
+	1    3350 5150
+	0    -1   -1   0
+$EndComp
+Wire Wire Line
+	3600 5300 5150 5300
+Wire Wire Line
+	5150 5300 5150 5650
+NoConn ~ 4950 5300
+Wire Wire Line
+	3600 5300 2200 5300
+Connection ~ 3600 5300
+Wire Wire Line
+	2200 5300 2200 5650
 $EndSCHEMATC

Commit message: Rev B
Parts:
- added TP21, TP22, TP23, TP24, TP25, TP26, TP27, TP28, TP29, TP30, TP31, TP32: TestPoint, symbol Connector:TestPoint
- C10, C11, C8, C9: DigiKey (none) -> 399-1100-1-ND
- J10, J11, J12, J9: DigiKey (none) -> 277-1247-ND
- U10, U8: DigiKey (none) -> 296-21928-1-ND
Other:
- note added: "(just for digikey)"
- note added: "Motor Driver Connectors"
Changed lines of the file:
@@
 F 2 "Package_SO:SOIC-14_3.9x8.7mm_P1.27mm" H 2100 5750 50  0001 C CNN
 F 3 "http://www.ti.com/lit/ds/symlink/txb0104.pdf" H 2210 6595 50  0001 C CNN
+F 4 "296-21928-1-ND" H 2100 6500 50  0001 C CNN "DigiKey"
 	1    2100 6500
 	1    0    0    -1
@@
 F 2 "Capacitor_SMD:C_0603_1608Metric_Pad1.05x0.95mm_HandSolder" H 1900 5650 50  0001 C CNN
 F 3 "~" H 1900 5650 50  0001 C CNN
+F 4 "399-1100-1-ND" H 1900 5650 50  0001 C CNN "DigiKey"
 	1    1900 5650
 	0    1    1    0
@@
 F 2 "Capacitor_SMD:C_0603_1608Metric_Pad1.05x0.95mm_HandSolder" H 2300 5650 50  0001 C CNN
 F 3 "~" H 2300 5650 50  0001 C CNN
+F 4 "399-1100-1-ND" H 2300 5650 50  0001 C CNN "DigiKey"
 	1    2300 5650
 	0    1    1    0
@@
 F 2 "Package_SO:SOIC-14_3.9x8.7mm_P1.27mm" H 5050 5750 50  0001 C CNN
 F 3 "http://www.ti.com/lit/ds/symlink/txb0104.pdf" H 5160 6595 50  0001 C CNN
+F 4 "296-21928-1-ND" H 5050 6500 50  0001 C CNN "DigiKey"
 	1    5050 6500
 	1    0    0    -1
@@
 F 2 "Capacitor_SMD:C_0603_1608Metric_Pad1.05x0.95mm_HandSolder" H 4850 5650 50  0001 C CNN
 F 3 "~" H 4850 5650 50  0001 C CNN
+F 4 "399-1100-1-ND" H 4850 5650 50  0001 C CNN "DigiKey"
 	1    4850 5650
 	0    1    1    0
@@
 F 2 "Capacitor_SMD:C_0603_1608Metric_Pad1.05x0.95mm_HandSolder" H 5250 5650 50  0001 C CNN
 F 3 "~" H 5250 5650 50  0001 C CNN
+F 4 "399-1100-1-ND" H 5250 5650 50  0001 C CNN "DigiKey"
 	1    5250 5650
 	0    1    1    0
@@
 F 2 "TerminalBlock_Phoenix:TerminalBlock_Phoenix_MKDS-3-2-5.08_1x02_P5.08mm_Horizontal" H 1200 1050 50  0001 C CNN
 F 3 "~" H 1200 1050 50  0001 C CNN
+F 4 "277-1247-ND" H 1200 1050 50  0001 C CNN "DigiKey"
 	1    1200 1050
 	0    -1   -1   0
@@
 F 2 "TerminalBlock_Phoenix:TerminalBlock_Phoenix_MKDS-3-2-5.08_1x02_P5.08mm_Horizontal" H 1200 1850 50  0001 C CNN
 F 3 "~" H 1200 1850 50  0001 C CNN
+F 4 "277-1247-ND" H 1200 1850 50  0001 C CNN "DigiKey"
 	1    1200 1850
 	0    -1   -1   0
@@
 F 2 "TerminalBlock_Phoenix:TerminalBlock_Phoenix_MKDS-3-2-5.08_1x02_P5.08mm_Horizontal" H 1200 2650 50  0001 C CNN
 F 3 "~" H 1200 2650 50  0001 C CNN
+F 4 "277-1247-ND" H 1200 2650 50  0001 C CNN "DigiKey"
 	1    1200 2650
 	0    -1   -1   0
@@
 F 2 "TerminalBlock_Phoenix:TerminalBlock_Phoenix_MKDS-3-2-5.08_1x02_P5.08mm_Horizontal" H 1200 3450 50  0001 C CNN
 F 3 "~" H 1200 3450 50  0001 C CNN
+F 4 "277-1247-ND" H 1200 3450 50  0001 C CNN "DigiKey"
 	1    1200 3450
 	0    -1   -1   0
@@
 Wire Wire Line
 	2200 5300 2200 5650
+$Comp
+L Connector:TestPoint TP21
+U 1 1 5EF090F9
+P 850 4500
+F 0 "TP21" H 908 4618 50  0000 L CNN
+F 1 "TestPoint" H 908 4527 50  0000 L CNN
+F 2 "" H 1050 4500 50  0001 C CNN
+F 3 "~" H 1050 4500 50  0001 C CNN
+F 4 "S7043-ND" H 850 4500 50  0001 C CNN "DigiKey"
+	1    850  4500
+	1    0    0    -1
+$EndComp
+$Comp
+L Connector:TestPoint TP23
+U 1 1 5EF09D1C
+P 950 4500
+F 0 "TP23" H 1008 4618 50  0000 L CNN
+F 1 "TestPoint" H 1008 4527 50  0000 L CNN
+F 2 "" H 1150 4500 50  0001 C CNN
+F 3 "~" H 1150 4500 50  0001 C CNN
+F 4 "S7043-ND" H 950 4500 50  0001 C CNN "DigiKey"
+	1    950  4500
+	1    0    0    -1
+$EndComp
+$Comp
+L Connector:TestPoint TP25
+U 1 1 5EF09F5F
+P 1050 4500
+F 0 "TP25" H 1108 4618 50  0000 L CNN
+F 1 "TestPoint" H 1108 4527 50  0000 L CNN
+F 2 "" H 1250 4500 50  0001 C CNN
+F 3 "~" H 1250 4500 50  0001 C CNN
+F 4 "S7043-ND" H 1050 4500 50  0001 C CNN "DigiKey"
+	1    1050 4500
+	1    0    0    -1
+$EndComp
+$Comp
+L Connector:TestPoint TP27
+U 1 1 5EF0A180
+P 1150 4500
+F 0 "TP27" H 1208 4618 50  0000 L CNN
+F 1 "TestPoint" H 1208 4527 50  0000 L CNN
+F 2 "" H 1350 4500 50  0001 C CNN
+F 3 "~" H 1350 4500 50  0001 C CNN
+F 4 "S7043-ND" H 1150 4500 50  0001 C CNN "DigiKey"
+	1    1150 4500
+	1    0    0    -1
+$EndComp
+$Comp
+L Connector:TestPoint TP22
+U 1 1 5EF0A47F
+P 850 4600
+F 0 "TP22" H 792 4626 50  0000 R CNN
+F 1 "TestPoint" H 792 4717 50  0000 R CNN
+F 2 "" H 1050 4600 50  0001 C CNN
+F 3 "~" H 1050 4600 50  0001 C CNN
+F 4 "S7041-ND" H 850 4600 50  0001 C CNN "DigiKey"
+	1    850  4600
+	-1   0    0    1
+$EndComp
+$Comp
+L Connector:TestPoint TP24
+U 1 1 5EF0AFA3
+P 950 4600
+F 0 "TP24" H 892 4626 50  0000 R CNN
+F 1 "TestPoint" H 892 4717 50  0000 R CNN
+F 2 "" H 1150 4600 50  0001 C CNN
+F 3 "~" H 1150 4600 50  0001 C CNN
+F 4 "S7041-ND" H 950 4600 50  0001 C CNN "DigiKey"
+	1    950  4600
+	-1   0    0    1
+$EndComp
+$Comp
+L Connector:TestPoint TP26
+U 1 1 5EF0B292
+P 1050 4600
+F 0 "TP26" H 992 4626 50  0000 R CNN
+F 1 "TestPoint" H 992 4717 50  0000 R CNN
+F 2 "" H 1250 4600 50  0001 C CNN
+F 3 "~" H 1250 4600 50  0001 C CNN
+F 4 "S7041-ND" H 1050 4600 50  0001 C CNN "DigiKey"
+	1    1050 4600
+	-1   0    0    1
+$EndComp
+$Comp
+L Connector:TestPoint TP28
+U 1 1 5EF0BE5F
+P 1150 4600
+F 0 "TP28" H 1092 4626 50  0000 R CNN
+F 1 "TestPoint" H 1092 4717 50  0000 R CNN
+F 2 "" H 1350 4600 50  0001 C CNN
+F 3 "~" H 1350 4600 50  0001 C CNN
+F 4 "S7041-ND" H 1150 4600 50  0001 C CNN "DigiKey"
+	1    1150 4600
+	-1   0    0    1
+$EndComp
+Text Notes 750  4300 0    50   ~ 0
+(just for digikey)
+Text Notes 600  4850 0    50   ~ 0
+Motor Driver Connectors
+$Comp
+L Connector:TestPoint TP29
+U 1 1 5EF0E1D1
+P 1750 4500
+F 0 "TP29" H 1808 4618 50  0000 L CNN
+F 1 "TestPoint" H 1808 4527 50  0000 L CNN
+F 2 "" H 1950 4500 50  0001 C CNN
+F 3 "~" H 1950 4500 50  0001 C CNN
+F 4 "S7004-ND" H 1750 4500 50  0001 C CNN "DigiKey"
+	1    1750 4500
+	1    0    0    -1
+$EndComp
+$Comp
+L Connector:TestPoint TP30
+U 1 1 5EF16CF5
+P 1850 4500
+F 0 "TP30" H 1908 4618 50  0000 L CNN
+F 1 "TestPoint" H 1908 4527 50  0000 L CNN
+F 2 "" H 2050 4500 50  0001 C CNN
+F 3 "~" H 2050 4500 50  0001 C CNN
+F 4 "S7004-ND" H 1850 4500 50  0001 C CNN "DigiKey"
+	1    1850 4500
+	1    0    0    -1
+$EndComp
+$Comp
+L Connector:TestPoint TP31
+U 1 1 5EF16FB4
+P 1950 4500
+F 0 "TP31" H 2008 4618 50  0000 L CNN
+F 1 "TestPoint" H 2008 4527 50  0000 L CNN
+F 2 "" H 2150 4500 50  0001 C CNN
+F 3 "~" H 2150 4500 50  0001 C CNN
+F 4 "S7004-ND" H 1950 4500 50  0001 C CNN "DigiKey"
+	1    1950 4500
+	1    0    0    -1
+$EndComp
+$Comp
+L Connector:TestPoint TP32
+U 1 1 5EF172C1
+P 2050 4500
+F 0 "TP32" H 2108 4618 50  0000 L CNN
+F 1 "TestPoint" H 2108 4527 50  0000 L CNN
+F 2 "" H 2250 4500 50  0001 C CNN
+F 3 "~" H 2250 4500 50  0001 C CNN
+F 4 "S7004-ND" H 2050 4500 50  0001 C CNN "DigiKey"
+	1    2050 4500
+	1    0    0    -1
+$EndComp
 $EndSCHEMATC
