File: TeensyIO.sch (KiCad schematic (older format))
At the start: 19 parts, among them U16 ADC128D818, U17 REF3030, U18 MCP23017_SS

Commit message: RevB
Connections:
- net +3V3: now also JP11.1 (A); no longer JP11.3 (B)
- net GND: now also JP11.3 (B); no longer JP11.1 (A)
Changed lines of the file:
@@
 F 3 "~" H 7600 2450 50  0001 C CNN
 	1    7600 2450
-	1    0    0    -1
+	-1   0    0    -1
 $EndComp
 $Comp

Commit message: Rev B
Parts:
- C28, C31, C33: DigiKey (none) -> 478-8657-1-ND
- C29, C30, C34: DigiKey (none) -> 399-1100-1-ND
- C32: DigiKey (none) -> 399-7934-1-ND
- R58, R59, R60, R61, R62: DigiKey (none) -> RR08P4.7KDCT-ND
- U16: DigiKey (none) -> 296-41182-1-ND
- U17: DigiKey (none) -> 296-26323-1-ND
Changed lines of the file:
@@
 F 2 "Package_SO:TSSOP-16_4.4x5mm_P0.65mm" H 2350 2600 50  0001 C CIN
 F 3 "http://www.ti.com/lit/ds/symlink/adc128d818.pdf" H 2350 2600 50  0001 C CNN
+F 4 "296-41182-1-ND" H 2350 2600 50  0001 C CNN "DigiKey"
 	1    2350 2600
 	1    0    0    -1
@@
 F 2 "Capacitor_SMD:C_0603_1608Metric_Pad1.05x0.95mm_HandSolder" H 2450 1550 50  0001 C CNN
 F 3 "~" H 2450 1550 50  0001 C CNN
+F 4 "399-1100-1-ND" H 2450 1550 50  0001 C CNN "DigiKey"
 	1    2450 1550
 	0    1    1    0
@@
 F 2 "Capacitor_SMD:C_0603_1608Metric_Pad1.05x0.95mm_HandSolder" H 2450 1200 50  0001 C CNN
 F 3 "~" H 2450 1200 50  0001 C CNN
+F 4 "478-8657-1-ND" H 2450 1200 50  0001 C CNN "DigiKey"
 	1    2450 1200
 	0    -1   -1   0
@@
 F 2 "Resistor_SMD:R_0603_1608Metric_Pad1.05x0.95mm_HandSolder" H 3500 2000 50  0001 C CNN
 F 3 "~" H 3500 2000 50  0001 C CNN
+F 4 "RR08P4.7KDCT-ND" H 3500 2000 50  0001 C CNN "DigiKey"
 	1    3500 2000
 	-1   0    0    1
@@
 F 2 "Resistor_SMD:R_0603_1608Metric_Pad1.05x0.95mm_HandSolder" H 3500 1700 50  0001 C CNN
 F 3 "~" H 3500 1700 50  0001 C CNN
+F 4 "RR08P4.7KDCT-ND" H 3500 1700 50  0001 C CNN "DigiKey"
 	1    3500 1700
 	-1   0    0    1
@@
 F 2 "Package_TO_SOT_SMD:SOT-23" H 4850 1500 50  0001 C CIN
 F 3 "http://www.ti.com/lit/ds/symlink/ref3033.pdf" H 4950 1600 50  0001 C CIN
+F 4 "296-26323-1-ND" H 4850 1950 50  0001 C CNN "DigiKey"
 	1    4850 1950
 	0    1    1    0
@@
 F 2 "Capacitor_SMD:C_0603_1608Metric_Pad1.05x0.95mm_HandSolder" H 5250 1750 50  0001 C CNN
 F 3 "~" H 5250 1750 50  0001 C CNN
+F 4 "399-7934-1-ND" H 5250 1750 50  0001 C CNN "DigiKey"
 	1    5250 1750
 	-1   0    0    1
@@
 F 2 "Capacitor_SMD:C_0603_1608Metric_Pad1.05x0.95mm_HandSolder" H 5200 2300 50  0001 C CNN
 F 3 "~" H 5200 2300 50  0001 C CNN
+F 4 "399-1100-1-ND" H 5200 2300 50  0001 C CNN "DigiKey"
 	1    5200 2300
 	0    -1   -1   0
@@
 F 2 "Capacitor_SMD:C_0603_1608Metric_Pad1.05x0.95mm_HandSolder" H 5200 2700 50  0001 C CNN
 F 3 "~" H 5200 2700 50  0001 C CNN
+F 4 "478-8657-1-ND" H 5200 2700 50  0001 C CNN "DigiKey"
 	1    5200 2700
 	0    -1   -1   0
@@
 F 2 "Capacitor_SMD:C_0603_1608Metric_Pad1.05x0.95mm_HandSolder" H 9500 1600 50  0001 C CNN
 F 3 "~" H 9500 1600 50  0001 C CNN
+F 4 "399-1100-1-ND" H 9500 1600 50  0001 C CNN "DigiKey"
 	1    9500 1600
 	0    1    1    0
@@
 F 2 "Capacitor_SMD:C_0603_1608Metric_Pad1.05x0.95mm_HandSolder" H 9500 1250 50  0001 C CNN
 F 3 "~" H 9500 1250 50  0001 C CNN
+F 4 "478-8657-1-ND" H 9500 1250 50  0001 C CNN "DigiKey"
 	1    9500 1250
 	0    -1   -1   0
@@
 F 2 "Resistor_SMD:R_0603_1608Metric_Pad1.05x0.95mm_HandSolder" H 8350 1900 50  0001 C CNN
 F 3 "~" H 8350 1900 50  0001 C CNN
+F 4 "RR08P4.7KDCT-ND" H 8350 1900 50  0001 C CNN "DigiKey"
 	1    8350 1900
 	1    0    0    -1
@@
 F 2 "Resistor_SMD:R_0603_1608Metric_Pad1.05x0.95mm_HandSolder" H 8350 2200 50  0001 C CNN
 F 3 "~" H 8350 2200 50  0001 C CNN
+F 4 "RR08P4.7KDCT-ND" H 8350 2200 50  0001 C CNN "DigiKey"
 	1    8350 2200
 	1    0    0    -1
@@
 F 2 "Resistor_SMD:R_0603_1608Metric_Pad1.05x0.95mm_HandSolder" H 8500 2900 50  0001 C CNN
 F 3 "~" H 8500 2900 50  0001 C CNN
+F 4 "RR08P4.7KDCT-ND" H 8500 2900 50  0001 C CNN "DigiKey"
 	1    8500 2900
 	0    1    1    0
