File: TurtlebotController.sch (KiCad schematic (older format))
At the start: 12 parts

Commit message: Added fuses
Parts:
- added F?: Fuse, symbol Device:Fuse
Connections:
- net +3V3: now also U?.5 (VDD); no longer U?.4 (VIN)
- net +5V: now also F?.1; no longer JP?.2
- new net: F?.2, JP?.2
Other:
- moved on the sheet: C?
Changed lines of the file:
@@
 L power:+3.3V #PWR?
 U 1 1 5E063C5B
-P 10250 5100
-F 0 "#PWR?" H 10250 4950 50  0001 C CNN
-F 1 "+3.3V" V 10265 5228 50  0000 L CNN
-F 2 "" H 10250 5100 50  0001 C CNN
-F 3 "" H 10250 5100 50  0001 C CNN
-	1    10250 5100
+P 10250 5200
+F 0 "#PWR?" H 10250 5050 50  0001 C CNN
+F 1 "+3.3V" V 10265 5328 50  0000 L CNN
+F 2 "" H 10250 5200 50  0001 C CNN
+F 3 "" H 10250 5200 50  0001 C CNN
+	1    10250 5200
 	0    1    1    0
 $EndComp
@@
 L Device:C_Small C?
 U 1 1 5E079BC3
-P 10050 5200
-F 0 "C?" H 10142 5246 50  0000 L CNN
-F 1 "10uF" H 10142 5155 50  0000 L CNN
-F 2 "" H 10050 5200 50  0001 C CNN
-F 3 "~" H 10050 5200 50  0001 C CNN
-	1    10050 5200
+P 10050 5300
+F 0 "C?" H 10142 5346 50  0000 L CNN
+F 1 "10uF" H 10142 5255 50  0000 L CNN
+F 2 "" H 10050 5300 50  0001 C CNN
+F 3 "~" H 10050 5300 50  0001 C CNN
+	1    10050 5300
 	1    0    0    -1
 $EndComp
@@
 L Device:C_Small C?
 U 1 1 5E07B8E0
-P 9600 5200
-F 0 "C?" H 9692 5246 50  0000 L CNN
-F 1 "0.1uF" H 9692 5155 50  0000 L CNN
-F 2 "" H 9600 5200 50  0001 C CNN
-F 3 "~" H 9600 5200 50  0001 C CNN
-	1    9600 5200
+P 9600 5300
+F 0 "C?" H 9692 5346 50  0000 L CNN
+F 1 "0.1uF" H 9692 5255 50  0000 L CNN
+F 2 "" H 9600 5300 50  0001 C CNN
+F 3 "~" H 9600 5300 50  0001 C CNN
+	1    9600 5300
 	1    0    0    -1
 $EndComp
@@
 	9450 5000 9500 5000
 Wire Wire Line
-	9450 5100 9600 5100
-Wire Wire Line
-	9600 5100 10050 5100
-Connection ~ 9600 5100
-Wire Wire Line
-	10050 5100 10250 5100
-Connection ~ 10050 5100
+	9450 5200 9600 5200
+Wire Wire Line
+	9600 5200 10050 5200
+Connection ~ 9600 5200
+Wire Wire Line
+	10050 5200 10250 5200
+Connection ~ 10050 5200
 $Comp
 L power:GND #PWR?
 U 1 1 5E0A8BF3
-P 9600 5400
-F 0 "#PWR?" H 9600 5150 50  0001 C CNN
-F 1 "GND" H 9605 5227 50  0000 C CNN
-F 2 "" H 9600 5400 50  0001 C CNN
-F 3 "" H 9600 5400 50  0001 C CNN
-	1    9600 5400
-	1    0    0    -1
-$EndComp
-Wire Wire Line
-	10050 5300 9600 5300
-Wire Wire Line
-	9600 5300 9600 5400
-Connection ~ 9600 5300
+P 9600 5500
+F 0 "#PWR?" H 9600 5250 50  0001 C CNN
+F 1 "GND" H 9605 5327 50  0000 C CNN
+F 2 "" H 9600 5500 50  0001 C CNN
+F 3 "" H 9600 5500 50  0001 C CNN
+	1    9600 5500
+	1    0    0    -1
+$EndComp
+Wire Wire Line
+	10050 5400 9600 5400
+Wire Wire Line
+	9600 5400 9600 5500
+Connection ~ 9600 5400
 $Sheet
 S 8100 2150 2150 1050
@@
 L power:+5V #PWR?
 U 1 1 5E126751
-P 5950 1150
-F 0 "#PWR?" H 5950 1000 50  0001 C CNN
-F 1 "+5V" H 5965 1323 50  0000 C CNN
-F 2 "" H 5950 1150 50  0001 C CNN
-F 3 "" H 5950 1150 50  0001 C CNN
-	1    5950 1150
+P 5950 850
+F 0 "#PWR?" H 5950 700 50  0001 C CNN
+F 1 "+5V" H 5965 1023 50  0000 C CNN
+F 2 "" H 5950 850 50  0001 C CNN
+F 3 "" H 5950 850 50  0001 C CNN
+	1    5950 850
 	1    0    0    -1
 $EndComp
@@
 Wire Wire Line
 	3850 3750 3950 3750
+$Comp
+L Device:Fuse F?
+U 1 1 5E2B6DA8
+P 5950 1000
+F 0 "F?" H 6010 1046 50  0000 L CNN
+F 1 "Fuse" H 6010 955 50  0000 L CNN
+F 2 "" V 5880 1000 50  0001 C CNN
+F 3 "~" H 5950 1000 50  0001 C CNN
+	1    5950 1000
+	1    0    0    -1
+$EndComp
 $EndSCHEMATC

Commit message: Added footprints
Parts:
- C1, C2: renamed from C?; footprint (none) -> Capacitor_SMD:C_0603_1608Metric_Pad1.05x0.95mm_HandSolder
- F1: renamed from F?; footprint (none) -> Fuse:Fuse_0805_2012Metric_Pad1.15x1.40mm_HandSolder
- J1: renamed from J?; footprint (none) -> Connector_PinHeader_2.54mm:PinHeader_2x20_P2.54mm_Vertical
- JP1, JP2, JP3: renamed from JP?; footprint (none) -> Jumper:SolderJumper-2_P1.3mm_Bridged_RoundedPad1.0x1.5mm
- JP4, JP5: renamed from JP?; footprint (none) -> Jumper:SolderJumper-2_P1.3mm_Open_RoundedPad1.0x1.5mm
- R1, R2: renamed from R?; footprint (none) -> Resistor_SMD:R_0603_1608Metric_Pad1.05x0.95mm_HandSolder
- U1: renamed from U?; footprint (none) -> teensy:Teensy40
- U2: renamed from U?; footprint (none) -> TurtlebotController:Pololu_MinIMU-9
Connections:
- net LEFT_ENCODER_A_3.3V: now also U1.6 (4_BCLK2); no longer U1.27 (20_A6_TX5_LRCLK1)
- net LEFT_ENCODER_B_3.3V: now also U1.7 (5_IN2); no longer U1.28 (21_A7_RX5_BCLK1)
- net LEFT_MOTOR_DIAGA: now also U1.27 (20_A6_TX5_LRCLK1); no longer U1.6 (4_BCLK2)
- net LEFT_MOTOR_DIAGB: now also U1.28 (21_A7_RX5_BCLK1); no longer U1.7 (5_IN2)
- net LEFT_MOTOR_PWM: now also U1.21 (14_A0_TX3_SPDIF_OUT); no longer U1.4 (2_OUT2)
- net RIGHT_ENCODER_A_3.3V: now also U1.4 (2_OUT2); no longer U1.21 (14_A0_TX3_SPDIF_OUT)
- net RIGHT_ENCODER_B_3.3V: now also U1.5 (3_LRCLK2); no longer U1.22 (15_A1_RX3_SPDIF_IN)
- net RIGHT_MOTOR_PWM: now also U1.22 (15_A1_RX3_SPDIF_IN); no longer U1.5 (3_LRCLK2)

Commit message: Added BOM
Parts:
- added U7: UltimateSensorFusion_MPU9250_PeskyProducts, TurtlebotController:UltimateSensorFusion_MPU9250, symbol pololu_parts:UltimateSensorFusion_MPU9250_PeskyProducts
- J1: DigiKey (none) -> 1528-1785-ND
- U1: DigiKey (none) -> 1568-DEV-15583-ND
Connections:
- net +3V3: now also U7.2 (3V3)
- net GND: now also U7.1 (GND)
- net SCL_0: now also U7.4 (SCL)
- net SDA_0: now also U7.5 (SDA)
- net TEENSY_HEARTBEAT: now also U1.3 (1_TX1_CTX2); no longer U1.29 (22_A8_CTX1)
- net MPU_INTERRUPT: now reaches U1.2 (0_RX1_CRX2)
- net MPU_INTERRUPT: now also U7.10 (INT)
- new net CURRENT_OUT: U1.29 (22_A8_CTX1)
Changed lines of the file:
@@
 F 2 "teensy:Teensy40" H 2350 2700 50  0001 C CNN
 F 3 "" H 2350 2700 50  0001 C CNN
+F 4 " 1568-DEV-15583-ND" H 2750 2500 50  0001 C CNN "DigiKey"
 	1    2750 2500
 	1    0    0    -1
@@
 F 2 "Connector_PinHeader_2.54mm:PinHeader_2x20_P2.54mm_Vertical" H 6100 3050 50  0001 C CNN
 F 3 "https://www.raspberrypi.org/documentation/hardware/raspberrypi/schematics/rpi_SCH_3bplus_1p0_reduced.pdf" H 6100 3050 50  0001 C CNN
+F 4 " 1528-1785-ND " H 6100 3050 50  0001 C CNN "DigiKey"
 	1    6100 3050
 	1    0    0    -1
@@
 Wire Wire Line
 	7000 3750 6900 3750
-Text GLabel 3950 3850 2    50   Input ~ 0
+Text GLabel 1650 1350 0    50   Input ~ 0
 TEENSY_HEARTBEAT
 Wire Wire Line
@@
 	1    0    0    -1
 $EndComp
+Text GLabel 3950 3850 2    50   Input ~ 0
+CURRENT_OUT
+$Comp
+L pololu_parts:UltimateSensorFusion_MPU9250_PeskyProducts U7
+U 1 1 5DFB05EC
+P 6300 5650
+F 0 "U7" H 6275 6175 50  0000 C CNN
+F 1 "UltimateSensorFusion_MPU9250_PeskyProducts" H 6275 6084 50  0000 C CNN
+F 2 "TurtlebotController:UltimateSensorFusion_MPU9250" H 6300 5650 50  0001 C CNN
+F 3 "" H 6300 5650 50  0001 C CNN
+	1    6300 5650
+	1    0    0    -1
+$EndComp
+Text GLabel 5850 5350 0    50   Input ~ 0
+SCL_0
+Text GLabel 5850 5450 0    50   Input ~ 0
+SDA_0
+Text GLabel 1650 1250 0    50   Input ~ 0
+MPU_INTERRUPT
+Text GLabel 5850 5550 0    50   Input ~ 0
+MPU_INTERRUPT
+$Comp
+L power:GND #PWR0171
+U 1 1 5DFCDA8F
+P 6700 5350
+F 0 "#PWR0171" H 6700 5100 50  0001 C CNN
+F 1 "GND" V 6705 5222 50  0000 R CNN
+F 2 "" H 6700 5350 50  0001 C CNN
+F 3 "" H 6700 5350 50  0001 C CNN
+	1    6700 5350
+	0    -1   -1   0
+$EndComp
+$Comp
+L power:+3.3V #PWR0172
+U 1 1 5DFCE474
+P 6950 5450
+F 0 "#PWR0172" H 6950 5300 50  0001 C CNN
+F 1 "+3.3V" H 6965 5623 50  0000 C CNN
+F 2 "" H 6950 5450 50  0001 C CNN
+F 3 "" H 6950 5450 50  0001 C CNN
+	1    6950 5450
+	0    1    1    0
+$EndComp
+Wire Wire Line
+	6950 5450 6700 5450
 $EndSCHEMATC

Commit message: Some fixes
Connections:
- net TEENSY_HEARTBEAT: now also U1.20 (13_SCK_CRX1_LED); no longer U1.3 (1_TX1_CTX2)
- net TEENSY_SCK: now also U1.3 (1_TX1_CTX2); no longer U1.20 (13_SCK_CRX1_LED)
- net LEFT_MOTOR_DIAGA renamed LEFT_MOTOR_INA
- net LEFT_MOTOR_DIAGB renamed LEFT_MOTOR_INB
- net RIGHT_MOTOR_DIAGA renamed RIGHT_MOTOR_INA
- net RIGHT_MOTOR_DIAGB renamed RIGHT_MOTOR_INB
Changed lines of the file:
@@
 	1600 3450 1650 3450
 Text GLabel 1600 3750 0    50   Input ~ 0
-LEFT_MOTOR_DIAGA
+LEFT_MOTOR_INA
 Text GLabel 1600 3850 0    50   Input ~ 0
-LEFT_MOTOR_DIAGB
+LEFT_MOTOR_INB
 Text GLabel 1600 1850 0    50   Input ~ 0
-RIGHT_MOTOR_DIAGA
+RIGHT_MOTOR_INA
 Text GLabel 1600 2150 0    50   Input ~ 0
-RIGHT_MOTOR_DIAGB
+RIGHT_MOTOR_INB
 Wire Wire Line
 	1600 1650 1650 1650
@@
 Wire Wire Line
 	1600 2250 1650 2250
-Text GLabel 1600 3050 0    50   Input ~ 0
+Text GLabel 1650 1350 0    50   Input ~ 0
 TEENSY_SCK
 Wire Wire Line
@@
 Wire Wire Line
 	7000 3750 6900 3750
-Text GLabel 1650 1350 0    50   Input ~ 0
+Text GLabel 1600 3050 0    50   Input ~ 0
 TEENSY_HEARTBEAT
 Wire Wire Line

Commit message: Most of rev B
Parts:
- added TP17: TestPoint, Connector_Wire:SolderWirePad_1x01_Drill1.2mm, symbol Connector:TestPoint
Connections:
- net LEFT_MOTOR_INA is gone; now on net TEENSY_TX: U1.27 (20_A6_TX5_LRCLK1)
- net LEFT_MOTOR_INB is gone; now on net TEENSY_RX: U1.28 (21_A7_RX5_BCLK1)
- net MPU_INTERRUPT: now also U1.13 (11_MOSI_CTX1); no longer U1.2 (0_RX1_CRX2)
- net TEENSY_CS: no longer U1.12 (10_CS_MQSR)
- net TEENSY_MISO: no longer U1.14 (12_MISO_MQSL)
- net TEENSY_MOSI: no longer U1.13 (11_MOSI_CTX1)
- net TEENSY_RX: no longer U1.9 (7_RX2_OUT1A)
- net TEENSY_SCK: no longer U1.3 (1_TX1_CTX2)
- net TEENSY_TX: no longer U1.10 (8_TX2_IN1)
- net MOTOR_4_ENCODER_B: now reaches U1.~ (GND)
- net MOTOR_4_ENCODER_B: now also TP17.1
- net LEFT_ENCODER_A_3.3V renamed MOTOR_3_ENCODER_A
- net LEFT_ENCODER_B_3.3V renamed MOTOR_3_ENCODER_B
- net LEFT_MOTOR_CURRENT renamed MOTOR_2_CS
- net LEFT_MOTOR_PWM renamed MOTOR_4_CS
- net RIGHT_ENCODER_A_3.3V renamed MOTOR_2_ENCODER_A
- net RIGHT_ENCODER_B_3.3V renamed MOTOR_2_ENCODER_B
- net RIGHT_MOTOR_CURRENT renamed MOTOR_1_CS
- net RIGHT_MOTOR_INA renamed MOTOR_1_PWM
- net RIGHT_MOTOR_INB renamed MOTOR_3_PWM
- net RIGHT_MOTOR_PWM renamed MOTOR_3_CS
- new net MOTOR_1_ENCODER_A: U1.2 (0_RX1_CRX2)
- new net MOTOR_1_ENCODER_B: U1.3 (1_TX1_CTX2)
- new net MOTOR_2_PWM: U1.10 (8_TX2_IN1)
- new net MOTOR_4_ENCODER_A: U1.9 (7_RX2_OUT1A)
- new net MOTOR_4_PWM: U1.12 (10_CS_MQSR)
- new net TEENSY_DEBUG: U1.14 (12_MISO_MQSL)
Other:
- moved on the sheet: JP1, JP2
Changed lines of the file:
@@
 $Descr A4 11693 8268
 encoding utf-8
-Sheet 1 4
+Sheet 1 6
 Title ""
 Date ""
@@
 Wire Wire Line
 	1550 2650 1650 2650
-Text GLabel 1600 3150 0    50   Input ~ 0
-LEFT_MOTOR_PWM
-Text GLabel 1600 3250 0    50   Input ~ 0
-RIGHT_MOTOR_PWM
 Wire Wire Line
 	1600 1450 1650 1450
 Wire Wire Line
 	1600 1550 1650 1550
-Text GLabel 1600 1650 0    50   Input ~ 0
-LEFT_ENCODER_A_3.3V
-Text GLabel 1600 1750 0    50   Input ~ 0
-LEFT_ENCODER_B_3.3V
 Wire Wire Line
 	1600 3850 1650 3850
 Wire Wire Line
 	1600 3750 1650 3750
-Text GLabel 1600 1550 0    50   Input ~ 0
-RIGHT_ENCODER_B_3.3V
-Text GLabel 1600 1450 0    50   Input ~ 0
-RIGHT_ENCODER_A_3.3V
 Wire Wire Line
 	1600 3150 1650 3150
 Wire Wire Line
 	1600 3250 1650 3250
-Text GLabel 1600 3350 0    50   Input ~ 0
-LEFT_MOTOR_CURRENT
-Text GLabel 1600 3450 0    50   Input ~ 0
-RIGHT_MOTOR_CURRENT
 Wire Wire Line
 	1600 3350 1650 3350
 Wire Wire Line
 	1600 3450 1650 3450
-Text GLabel 1600 3750 0    50   Input ~ 0
-LEFT_MOTOR_INA
-Text GLabel 1600 3850 0    50   Input ~ 0
-LEFT_MOTOR_INB
-Text GLabel 1600 1850 0    50   Input ~ 0
-RIGHT_MOTOR_INA
-Text GLabel 1600 2150 0    50   Input ~ 0
-RIGHT_MOTOR_INB
 Wire Wire Line
 	1600 1650 1650 1650
 Wire Wire Line
 	1600 1750 1650 1750
-Wire Wire Line
-	1600 1850 1650 1850
 $Comp
 L pololu_parts:MinIMU-9_V5 U2
@@
 Wire Wire Line
 	1600 2150 1650 2150
-Text GLabel 1600 1950 0    50   Input ~ 0
+Text GLabel 1600 3850 0    50   Input ~ 0
 TEENSY_RX
-Text GLabel 1600 2050 0    50   Input ~ 0
+Text GLabel 1600 3750 0    50   Input ~ 0
 TEENSY_TX
 Wire Wire Line
@@
 Wire Wire Line
 	5250 2150 5300 2150
-Text GLabel 1600 2250 0    50   Input ~ 0
-TEENSY_CS
-Text GLabel 1600 2350 0    50   Input ~ 0
-TEENSY_MOSI
-Text GLabel 1600 2450 0    50   Input ~ 0
-TEENSY_MISO
 Wire Wire Line
 	1600 2450 1650 2450
@@
 Wire Wire Line
 	1600 2250 1650 2250
-Text GLabel 1650 1350 0    50   Input ~ 0
-TEENSY_SCK
 Wire Wire Line
 	1600 3050 1650 3050
@@
 	8150 5150 8400 5150
 Connection ~ 8400 5150
-Text GLabel 950  3550 0    50   Input ~ 0
+Text GLabel 800  3550 0    50   Input ~ 0
 SDA_0
-Text GLabel 950  3650 0    50   Input ~ 0
+Text GLabel 800  3650 0    50   Input ~ 0
 SCL_0
 $Comp
@@
 L Device:Jumper_NC_Small JP2
 U 1 1 5E207A97
-P 1450 3650
-F 0 "JP2" H 1450 3862 50  0000 C CNN
-F 1 "SCL_TEENSY" H 1450 3771 50  0000 C CNN
-F 2 "Jumper:SolderJumper-2_P1.3mm_Bridged_RoundedPad1.0x1.5mm" H 1450 3650 50  0001 C CNN
-F 3 "~" H 1450 3650 50  0001 C CNN
-	1    1450 3650
-	1    0    0    -1
-$EndComp
-Wire Wire Line
-	950  3550 1000 3550
-Wire Wire Line
-	1200 3550 1650 3550
-Wire Wire Line
-	950  3650 1350 3650
-Wire Wire Line
-	1550 3650 1650 3650
+P 900 3650
+F 0 "JP2" H 900 3450 50  0000 C CNN
+F 1 "SCL_TEENSY" H 850 3550 50  0000 C CNN
+F 2 "Jumper:SolderJumper-2_P1.3mm_Bridged_RoundedPad1.0x1.5mm" H 900 3650 50  0001 C CNN
+F 3 "~" H 900 3650 50  0001 C CNN
+	1    900  3650
+	1    0    0    -1
+$EndComp
 $Comp
 L Device:Jumper_NC_Small JP1
 U 1 1 5E207299
-P 1100 3550
-F 0 "JP1" H 1100 3762 50  0000 C CNN
-F 1 "SDA_TEENSY" H 1100 3671 50  0000 C CNN
-F 2 "Jumper:SolderJumper-2_P1.3mm_Bridged_RoundedPad1.0x1.5mm" H 1100 3550 50  0001 C CNN
-F 3 "~" H 1100 3550 50  0001 C CNN
-	1    1100 3550
+P 900 3550
+F 0 "JP1" H 900 3762 50  0000 C CNN
+F 1 "SDA_TEENSY" H 900 3671 50  0000 C CNN
+F 2 "Jumper:SolderJumper-2_P1.3mm_Bridged_RoundedPad1.0x1.5mm" H 900 3550 50  0001 C CNN
+F 3 "~" H 900 3550 50  0001 C CNN
+	1    900  3550
 	1    0    0    -1
 $EndComp
@@
 F1 "Power.sch" 50
 $EndSheet
-Text GLabel 3950 3750 2    50   Input ~ 0
-BAT_VOLTAGE
 Wire Wire Line
 	3850 3750 3950 3750
@@
 	1    0    0    -1
 $EndComp
-Text GLabel 3950 3850 2    50   Input ~ 0
-CURRENT_OUT
 $Comp
 L pololu_parts:UltimateSensorFusion_MPU9250_PeskyProducts U7
@@
 Text GLabel 5850 5450 0    50   Input ~ 0
 SDA_0
-Text GLabel 1650 1250 0    50   Input ~ 0
+Text GLabel 1600 2350 0    50   Input ~ 0
 MPU_INTERRUPT
 Text GLabel 5850 5550 0    50   Input ~ 0
@@
 Wire Wire Line
 	6950 5450 6700 5450
+$Sheet
+S 4250 6300 2400 1250
+U 5ED727AE
+F0 "TeensyIO" 50
+F1 "TeensyIO.sch" 50
+$EndSheet
+Text GLabel 1600 1650 0    50   Input ~ 0
+MOTOR_3_ENCODER_A
+Text GLabel 1600 1750 0    50   Input ~ 0
+MOTOR_3_ENCODER_B
+Text GLabel 4100 2450 2    50   Input ~ 0
+MOTOR_4_ENCODER_B
+Text GLabel 1600 1950 0    50   Input ~ 0
+MOTOR_4_ENCODER_A
+Text GLabel 1600 1250 0    50   Input ~ 0
+MOTOR_1_ENCODER_A
+Text GLabel 1600 1350 0    50   Input ~ 0
+MOTOR_1_ENCODER_B
+Text GLabel 1600 1550 0    50   Input ~ 0
+MOTOR_2_ENCODER_B
+Text GLabel 1600 1450 0    50   Input ~ 0
+MOTOR_2_ENCODER_A
+Wire Wire Line
+	3850 2450 4050 2450
+$Comp
+L Connector:TestPoint TP17
+U 1 1 5F21F998
+P 4050 2550
+F 0 "TP17" H 3992 2576 50  0000 R CNN
+F 1 "TestPoint" H 3992 2667 50  0000 R CNN
+F 2 "Connector_Wire:SolderWirePad_1x01_Drill1.2mm" H 4250 2550 50  0001 C CNN
+F 3 "~" H 4250 2550 50  0001 C CNN
+	1    4050 2550
+	-1   0    0    1
+$EndComp
+Wire Wire Line
+	4050 2550 4050 2450
+Connection ~ 4050 2450
+Wire Wire Line
+	4050 2450 4100 2450
+Wire Wire Line
+	1600 1250 1650 1250
+Wire Wire Line
+	1600 1350 1650 1350
+Text GLabel 1600 2250 0    50   Input ~ 0
+MOTOR_4_PWM
+Text GLabel 1600 2050 0    50   Input ~ 0
+MOTOR_2_PWM
+Text GLabel 1600 2150 0    50   Input ~ 0
+MOTOR_3_PWM
+Text GLabel 1600 1850 0    50   Input ~ 0
+MOTOR_1_PWM
+Wire Wire Line
+	1600 1850 1650 1850
+Text GLabel 3950 3750 2    50   Input ~ 0
+BAT_VOLTAGE
+Text GLabel 3950 3850 2    50   Input ~ 0
+CURRENT_OUT
+Text GLabel 1600 3350 0    50   Output ~ 0
+MOTOR_2_CS
+Text GLabel 1600 3450 0    50   Output ~ 0
+MOTOR_1_CS
+Text GLabel 1600 3150 0    50   Output ~ 0
+MOTOR_4_CS
+Text GLabel 1600 3250 0    50   Output ~ 0
+MOTOR_3_CS
+Wire Wire Line
+	1000 3650 1650 3650
+Wire Wire Line
+	1650 3550 1000 3550
+Text GLabel 1600 2450 0    50   Input ~ 0
+TEENSY_DEBUG
 $EndSCHEMATC

Commit message: Rev B
Parts:
- added TP18, TP19, TP20: TestPoint, symbol Connector:TestPoint
- C2: DigiKey (none) -> 478-8646-1-ND
Other:
- note added: "(just for digikey)"
- note added: "Teensy Headers"
Changed lines of the file:
@@
 F 2 "Capacitor_SMD:C_0603_1608Metric_Pad1.05x0.95mm_HandSolder" H 10050 5300 50  0001 C CNN
 F 3 "~" H 10050 5300 50  0001 C CNN
+F 4 "478-8646-1-ND" H 10050 5300 50  0001 C CNN "DigiKey"
 	1    10050 5300
 	1    0    0    -1
@@
 Text GLabel 1600 2450 0    50   Input ~ 0
 TEENSY_DEBUG
+$Comp
+L Connector:TestPoint TP18
+U 1 1 5EEE1FF2
+P 950 5150
+F 0 "TP18" H 1008 5268 50  0000 L CNN
+F 1 "TestPoint" H 1008 5177 50  0000 L CNN
+F 2 "" H 1150 5150 50  0001 C CNN
+F 3 "~" H 1150 5150 50  0001 C CNN
+F 4 "S7047-ND" H 950 5150 50  0001 C CNN "DigiKey"
+	1    950  5150
+	1    0    0    -1
+$EndComp
+Text Notes 900  4900 0    50   ~ 0
+(just for digikey)
+$Comp
+L Connector:TestPoint TP19
+U 1 1 5EEE6208
+P 950 5200
+F 0 "TP19" H 892 5226 50  0000 R CNN
+F 1 "TestPoint" H 892 5317 50  0000 R CNN
+F 2 "" H 1150 5200 50  0001 C CNN
+F 3 "~" H 1150 5200 50  0001 C CNN
+F 4 "S7047-ND" H 950 5200 50  0001 C CNN "DigiKey"
+	1    950  5200
+	-1   0    0    1
+$EndComp
+$Comp
+L Connector:TestPoint TP20
+U 1 1 5EEE71EE
+P 1400 5150
+F 0 "TP20" H 1458 5268 50  0000 L CNN
+F 1 "TestPoint" H 1458 5177 50  0000 L CNN
+F 2 "" H 1600 5150 50  0001 C CNN
+F 3 "~" H 1600 5150 50  0001 C CNN
+F 4 "S7038-ND" H 1400 5150 50  0001 C CNN "DigiKey"
+	1    1400 5150
+	1    0    0    -1
+$EndComp
+Text Notes 950  5500 0    50   ~ 0
+Teensy Headers
 $EndSCHEMATC
