File: TurtlebotController.kicad_pcb (KiCad board)
At the start: 2 copper layers, 75 parts, among them J1 Raspberry_Pi_2_3, J2 LEFT_MOTOR, J3 RIGHT_MOTOR, J4 5V_OUT, J5 3.3V _OUT, J6 12V_OUT, U1 Teensy4.0, U2 MinIMU-9_V5, U3 VNH5019, U4 VNH5019, U5 ACS711xLCTR-25AB, U6 D24V90F5

Commit message: Added BOM
Parts:
- added REF**: MountingHole_4.3mm_M4_DIN965_Pad, MountingHole:MountingHole_4.3mm_M4_DIN965_Pad, F.Cu at (78.5, 111.4)
- added REF**: MountingHole_4.3mm_M4_DIN965_Pad, MountingHole:MountingHole_4.3mm_M4_DIN965_Pad, F.Cu at (174.5, 111.4)
- added REF**: MountingHole_4.3mm_M4_DIN965_Pad, MountingHole:MountingHole_4.3mm_M4_DIN965_Pad, F.Cu at (78.5, 45.4)
- added REF**: MountingHole_4.3mm_M4_DIN965_Pad, MountingHole:MountingHole_4.3mm_M4_DIN965_Pad, F.Cu at (174.5, 45.4)
- added U7: UltimateSensorFusion_MPU9250_PeskyProducts, TurtlebotController:UltimateSensorFusion_MPU9250, F.Cu at (116.5, 109.0)
- moved R18 116.5 mm to (108.8, 104.7), turned to 270 degrees
- moved U6 109.6 mm to (128.0, 49.9), turned to 90 degrees
- moved BT1 97.1 mm to (155.8, 44.4)
- moved J6 93.9 mm to (165.6, 114.4)
- moved C3 93.1 mm to (135.0, 49.2)
- moved U5 76.9 mm to (142.0, 45.9), turned to 180 degrees
- moved J5 73.8 mm to (158.7, 114.4)
- moved F4 73.3 mm to (148.5, 47.6)
- moved R1 71.5 mm to (122.4, 94.9), turned to 180 degrees
- moved R16 69.1 mm to (169.8, 91.7), turned to 270 degrees
- moved R2 66.8 mm to (122.4, 92.9)
- moved F3 65.8 mm to (169.0, 100.5), turned to 270 degrees
- moved F2 65.6 mm to (169.0, 71.5), turned to 270 degrees
- moved R19 64.8 mm to (135.9, 46.5), turned to 90 degrees
- moved R17 64.1 mm to (173.6, 97.9), turned to 180 degrees
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Connections:
- U1 pad 2: Net-(U1-Pad2) -> MPU_INTERRUPT
- U1 pad 29: TEENSY_HEARTBEAT -> CURRENT_OUT
- U1 pad 3: Net-(U1-Pad3) -> TEENSY_HEARTBEAT
Routing:
- net +12V: track 0.00 -> 278.6 mm, vias 0 -> 4
- net +5V: track 0.00 -> 262.1 mm, vias 0 -> 7
- net +3V3: track 0.00 -> 212.4 mm, vias 0 -> 8
- net RASPBERRY_3.3V: track 0.00 -> 115.3 mm, vias 0 -> 2
- net CURRENT_OUT: track 0.00 -> 102.1 mm, vias 0 -> 5
- net LEFT_ENCODER_B_3.3V: track 0.00 -> 101.4 mm, vias 0 -> 8
- net SCL_0: track 0.00 -> 101.3 mm, vias 0 -> 2
- net SDA_0: track 0.00 -> 99.8 mm, vias 0 -> 3
- net RASPBERRY_HEARTBEAT: track 0.00 -> 98.9 mm
- net LEFT_ENCODER_A_3.3V: track 0.00 -> 93.3 mm, vias 0 -> 6
- net TEENSY_TX: track 0.00 -> 89.3 mm, vias 0 -> 3
- net LEFT_MOTOR_DIAGA: track 0.00 -> 85.8 mm, vias 0 -> 5
- net LEFT_MOTOR_DIAGB: track 0.00 -> 79.0 mm, vias 0 -> 5
- net LEFT_MOTOR_CURRENT: track 0.00 -> 78.2 mm, vias 0 -> 4
- net RIGHT_ENCODER_B_3.3V: track 0.00 -> 76.8 mm, vias 0 -> 6
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- added copper zone on B.Cu, net GND
- added copper zone on F.Cu, net GND
Other:
- board outline added: 110 x 80 mm
- net class Power added: clearance 0.2, trace_width 0.5, via_dia 0.8, via_drill 0.4
- board text added: "- +"
- board text added: "Abiel Fernández TurtlebotController Rev. A 2019"

Commit message: Most of rev B
Parts:
- removed D7: LEFT_MOTOR_OK, LED_SMD:LED_0603_1608Metric_Pad1.05x0.95mm_HandSolder
- removed D8: RIGHT_MOTOR_OK, LED_SMD:LED_0603_1608Metric_Pad1.05x0.95mm_HandSolder
- removed F2, F3: Fuse, Fuse:Fuse_0805_2012Metric_Pad1.15x1.40mm_HandSolder
- removed R10, R9: 500Ohm, Resistor_SMD:R_0603_1608Metric_Pad1.05x0.95mm_HandSolder
- removed the REF** at (78.5, 111.4)
- removed the REF** at (174.5, 111.4)
- removed the REF** at (78.5, 45.4)
- removed the REF** at (174.5, 45.4)
- removed TP1: GND, TestPoint:TestPoint_Pad_D1.5mm
- removed TP10: RIGHT_ENCODER_B_5V, TestPoint:TestPoint_Pad_D1.5mm
- removed TP11: LEFT_PWM, TestPoint:TestPoint_Pad_D1.5mm
- removed TP12: RIGHT_ENCODER_A_3.3V, TestPoint:TestPoint_Pad_D1.5mm
- removed TP13: RIGHT_ENCODER_B_3.3V, TestPoint:TestPoint_Pad_D1.5mm
- removed TP14: RIGHT_PWM, TestPoint:TestPoint_Pad_D1.5mm
- removed TP2: LEFT_ENCODER_A_5V, TestPoint:TestPoint_Pad_D1.5mm
- removed TP3: LEFT_ENCODER_B_5V, TestPoint:TestPoint_Pad_D1.5mm
- removed TP7: LEFT_ENCODER_A_3.3V, TestPoint:TestPoint_Pad_D1.5mm
- removed TP8: LEFT_ENCODER_B_3.3V, TestPoint:TestPoint_Pad_D1.5mm
- removed TP9: RIGHT_ENCODER_A_5V, TestPoint:TestPoint_Pad_D1.5mm
- added C10: 0.1uF, Capacitor_SMD:C_0603_1608Metric_Pad1.05x0.95mm_HandSolder, F.Cu at (125.7, 90.7)
- added C11: 0.1uF, Capacitor_SMD:C_0603_1608Metric_Pad1.05x0.95mm_HandSolder, F.Cu at (129.5, 101.8)
- added C12: 33nF, Capacitor_SMD:C_0603_1608Metric_Pad1.05x0.95mm_HandSolder, F.Cu at (137.4, 80.5)
- added C13: 33nF, Capacitor_SMD:C_0603_1608Metric_Pad1.05x0.95mm_HandSolder, F.Cu at (137.9, 117.3)
- added C14: 0.1uF, Capacitor_SMD:C_0603_1608Metric_Pad1.05x0.95mm_HandSolder, F.Cu at (152.9, 80.4)
- added C15: 0.1uF, Capacitor_SMD:C_0603_1608Metric_Pad1.05x0.95mm_HandSolder, F.Cu at (152.8, 122.0)
- added C16: 47uF, Capacitor_Tantalum_SMD:CP_EIA-3216-10_Kemet-I_Pad1.58x1.35mm_HandSolder, F.Cu at (146.1, 56.7)
- added C17: 0.1uF, Capacitor_SMD:C_0603_1608Metric_Pad1.05x0.95mm_HandSolder, F.Cu at (146.9, 58.6)
- added C18: 47uF, Capacitor_Tantalum_SMD:CP_EIA-3216-10_Kemet-I_Pad1.58x1.35mm_HandSolder, F.Cu at (149.3, 99.4)
- added C19: 0.1uF, Capacitor_SMD:C_0603_1608Metric_Pad1.05x0.95mm_HandSolder, F.Cu at (148.6, 97.5)
- added C20: 33nF, Capacitor_SMD:C_0603_1608Metric_Pad1.05x0.95mm_HandSolder, F.Cu at (168.4, 77.0)
- added C21: 33nF, Capacitor_SMD:C_0603_1608Metric_Pad1.05x0.95mm_HandSolder, F.Cu at (169.2, 117.5)
- added C22: 0.1uF, Capacitor_SMD:C_0603_1608Metric_Pad1.05x0.95mm_HandSolder, F.Cu at (184.2, 79.8)
- added C23: 0.1uF, Capacitor_SMD:C_0603_1608Metric_Pad1.05x0.95mm_HandSolder, F.Cu at (184.2, 122.2)
- added C24: 47uF, Capacitor_Tantalum_SMD:CP_EIA-3216-10_Kemet-I_Pad1.58x1.35mm_HandSolder, F.Cu at (180.7, 57.6)
- added C25: 0.1uF, Capacitor_SMD:C_0603_1608Metric_Pad1.05x0.95mm_HandSolder, F.Cu at (180.2, 55.6)
- added C26: 47uF, Capacitor_Tantalum_SMD:CP_EIA-3216-10_Kemet-I_Pad1.58x1.35mm_HandSolder, F.Cu at (181.0, 99.5)
- added C27: 0.1uF, Capacitor_SMD:C_0603_1608Metric_Pad1.05x0.95mm_HandSolder, F.Cu at (180.2, 97.5)
- added C28: 1uF, Capacitor_SMD:C_0603_1608Metric_Pad1.05x0.95mm_HandSolder, F.Cu at (88.5, 85.3)
- added C29: 0.1uF, Capacitor_SMD:C_0603_1608Metric_Pad1.05x0.95mm_HandSolder, F.Cu at (88.5, 87.1)
- added C30: 0.1uF, Capacitor_SMD:C_0603_1608Metric_Pad1.05x0.95mm_HandSolder, F.Cu at (95.3, 85.3)
- added C31: 1uF, Capacitor_SMD:C_0603_1608Metric_Pad1.05x0.95mm_HandSolder, F.Cu at (95.3, 87.0)
- added C32: 0.47uF, Capacitor_SMD:C_0603_1608Metric_Pad1.05x0.95mm_HandSolder, F.Cu at (92.7, 82.6)
- added C33: 1uF, Capacitor_SMD:C_0603_1608Metric_Pad1.05x0.95mm_HandSolder, F.Cu at (119.3, 76.6)
- added C34: 0.1uF, Capacitor_SMD:C_0603_1608Metric_Pad1.05x0.95mm_HandSolder, F.Cu at (117.7, 76.6)
- added C8: 0.1uF, Capacitor_SMD:C_0603_1608Metric_Pad1.05x0.95mm_HandSolder, F.Cu at (125.5, 101.8)
- added C9: 0.1uF, Capacitor_SMD:C_0603_1608Metric_Pad1.05x0.95mm_HandSolder, F.Cu at (129.3, 90.8)
- added D10: LED_Dual_2pin, LED_SMD:LED_0603_1608Metric_Pad1.05x0.95mm_HandSolder, F.Cu at (160.2, 100.8)
- added D11: LED_Dual_2pin, LED_SMD:LED_0603_1608Metric_Pad1.05x0.95mm_HandSolder, F.Cu at (191.5, 57.2)
- added D12: LED_Dual_2pin, LED_SMD:LED_0603_1608Metric_Pad1.05x0.95mm_HandSolder, F.Cu at (191.0, 100.0)
- added D13: TEENSY_DEBUG, LED_SMD:LED_0603_1608Metric_Pad1.05x0.95mm_HandSolder, F.Cu at (81.5, 126.8)
- added D9: LED_Dual_2pin, LED_SMD:LED_0603_1608Metric_Pad1.05x0.95mm_HandSolder, F.Cu at (159.0, 57.7)
- added J10: Screw_Terminal_01x02, TerminalBlock_Phoenix:TerminalBlock_Phoenix_MKDS-3-2-5.08_1x02_P5.08mm_Horizontal, F.Cu at (210.5, 77.2)
- added J11: Screw_Terminal_01x02, TerminalBlock_Phoenix:TerminalBlock_Phoenix_MKDS-3-2-5.08_1x02_P5.08mm_Horizontal, F.Cu at (210.5, 104.8)
- added J12: Screw_Terminal_01x02, TerminalBlock_Phoenix:TerminalBlock_Phoenix_MKDS-3-2-5.08_1x02_P5.08mm_Horizontal, F.Cu at (210.5, 122.9)
- added J7: MOTOR_3, Connector_PinHeader_2.54mm:PinHeader_1x06_P2.54mm_Vertical, F.Cu at (200.5, 98.5)
- added J8: MOTOR_4, Connector_PinHeader_2.54mm:PinHeader_1x06_P2.54mm_Vertical, F.Cu at (200.5, 116.5)
- added J9: Screw_Terminal_01x02, TerminalBlock_Phoenix:TerminalBlock_Phoenix_MKDS-3-2-5.08_1x02_P5.08mm_Horizontal, F.Cu at (210.5, 59.3)
- added JP10: Jumper_3_Bridged12, Jumper:SolderJumper-3_P1.3mm_Bridged12_RoundedPad1.0x1.5mm, F.Cu at (113.3, 93.4)
- added JP11: Jumper_3_Bridged12, Jumper:SolderJumper-3_P1.3mm_Bridged12_RoundedPad1.0x1.5mm, F.Cu at (114.3, 97.4)
- added JP12: Jumper_3_Bridged12, Jumper:SolderJumper-3_P1.3mm_Bridged12_RoundedPad1.0x1.5mm, F.Cu at (110.5, 95.6)
- added JP13: Jumper_3_Bridged12, Jumper:SolderJumper-3_P1.3mm_Bridged12_RoundedPad1.0x1.5mm, F.Cu at (110.5, 90.8)
- added JP6: Jumper_3_Bridged12, Jumper:SolderJumper-3_P1.3mm_Bridged12_RoundedPad1.0x1.5mm, F.Cu at (196.8, 60.6)
- added JP7: Jumper_3_Bridged12, Jumper:SolderJumper-3_P1.3mm_Bridged12_RoundedPad1.0x1.5mm, F.Cu at (196.8, 106.1)
- added JP8: Jumper_3_Bridged12, Jumper:SolderJumper-3_P1.3mm_Bridged12_RoundedPad1.0x1.5mm, F.Cu at (196.8, 78.6)
- added JP9: Jumper_3_Bridged12, Jumper:SolderJumper-3_P1.3mm_Bridged12_RoundedPad1.0x1.5mm, F.Cu at (196.8, 124.1)
- added Q1: BUK7M12-40EX, Package_TO_SOT_SMD:LFPAK33, F.Cu at (137.0, 61.6)
- added Q2: BUK7M12-40EX, Package_TO_SOT_SMD:LFPAK33, F.Cu at (136.9, 103.0)
- added Q3: BUK7M12-40EX, Package_TO_SOT_SMD:LFPAK33, F.Cu at (168.2, 61.0)
- added Q4: BUK7M12-40EX, Package_TO_SOT_SMD:LFPAK33, F.Cu at (168.2, 103.1)
- added R22: 4.7k, Resistor_SMD:R_0603_1608Metric_Pad1.05x0.95mm_HandSolder, F.Cu at (142.4, 83.0)
- added R23: 4.7k, Resistor_SMD:R_0603_1608Metric_Pad1.05x0.95mm_HandSolder, F.Cu at (141.9, 125.1)
- added R24: 4.7k, Resistor_SMD:R_0603_1608Metric_Pad1.05x0.95mm_HandSolder, F.Cu at (148.6, 83.0)
- added R25: 4.7k, Resistor_SMD:R_0603_1608Metric_Pad1.05x0.95mm_HandSolder, F.Cu at (149.9, 125.1)
- added R26: 1k, Resistor_SMD:R_0603_1608Metric_Pad1.05x0.95mm_HandSolder, F.Cu at (137.4, 75.4)
- added R27: 1k, Resistor_SMD:R_0603_1608Metric_Pad1.05x0.95mm_HandSolder, F.Cu at (140.3, 125.1)
- added R28: 10k, Resistor_SMD:R_0603_1608Metric_Pad1.05x0.95mm_HandSolder, F.Cu at (138.3, 77.9)
- added R29: 10k, Resistor_SMD:R_0603_1608Metric_Pad1.05x0.95mm_HandSolder, F.Cu at (136.3, 117.3)
- added R30: 1k, Resistor_SMD:R_0603_1608Metric_Pad1.05x0.95mm_HandSolder, F.Cu at (150.2, 83.0)
- added R31: 1k, Resistor_SMD:R_0603_1608Metric_Pad1.05x0.95mm_HandSolder, F.Cu at (136.6, 77.9)
- added R32: 1k, Resistor_SMD:R_0603_1608Metric_Pad1.05x0.95mm_HandSolder, F.Cu at (151.5, 125.1)
- added R33: 1k, Resistor_SMD:R_0603_1608Metric_Pad1.05x0.95mm_HandSolder, F.Cu at (137.1, 114.8)
- added R34: 4.7k, Resistor_SMD:R_0603_1608Metric_Pad1.05x0.95mm_HandSolder, F.Cu at (159.0, 59.3)
- added R35: 4.7k, Resistor_SMD:R_0603_1608Metric_Pad1.05x0.95mm_HandSolder, F.Cu at (160.2, 102.4)
- added R36: 1k, Resistor_SMD:R_0603_1608Metric_Pad1.05x0.95mm_HandSolder, F.Cu at (173.9, 83.3)
- added R37: 1k, Resistor_SMD:R_0603_1608Metric_Pad1.05x0.95mm_HandSolder, F.Cu at (181.9, 83.3)
- added R38: 1k, Resistor_SMD:R_0603_1608Metric_Pad1.05x0.95mm_HandSolder, F.Cu at (174.0, 125.5)
- added R39: 1k, Resistor_SMD:R_0603_1608Metric_Pad1.05x0.95mm_HandSolder, F.Cu at (181.0, 125.5)
- added R40: 1k, Resistor_SMD:R_0603_1608Metric_Pad1.05x0.95mm_HandSolder, F.Cu at (177.1, 83.3)
- added R41: 1k, Resistor_SMD:R_0603_1608Metric_Pad1.05x0.95mm_HandSolder, F.Cu at (177.5, 125.5)
- added R42: 10k, Resistor_SMD:R_0603_1608Metric_Pad1.05x0.95mm_HandSolder, F.Cu at (178.7, 83.3)
- added R43: 10k, Resistor_SMD:R_0603_1608Metric_Pad1.05x0.95mm_HandSolder, F.Cu at (179.2, 125.5)
- added R44: 4.7k, Resistor_SMD:R_0603_1608Metric_Pad1.05x0.95mm_HandSolder, F.Cu at (175.5, 83.3)
- added R45: 4.7k, Resistor_SMD:R_0603_1608Metric_Pad1.05x0.95mm_HandSolder, F.Cu at (175.8, 125.5)
- added R46: 4.7k, Resistor_SMD:R_0603_1608Metric_Pad1.05x0.95mm_HandSolder, F.Cu at (180.3, 83.3)
- added R47: 4.7k, Resistor_SMD:R_0603_1608Metric_Pad1.05x0.95mm_HandSolder, F.Cu at (182.8, 125.5)
- added R48: 1k, Resistor_SMD:R_0603_1608Metric_Pad1.05x0.95mm_HandSolder, F.Cu at (172.3, 83.3)
- added R49: 1k, Resistor_SMD:R_0603_1608Metric_Pad1.05x0.95mm_HandSolder, F.Cu at (172.2, 125.5)
- added R50: 10k, Resistor_SMD:R_0603_1608Metric_Pad1.05x0.95mm_HandSolder, F.Cu at (167.5, 74.4)
- added R51: 10k, Resistor_SMD:R_0603_1608Metric_Pad1.05x0.95mm_HandSolder, F.Cu at (167.5, 117.5)
- added R52: 1k, Resistor_SMD:R_0603_1608Metric_Pad1.05x0.95mm_HandSolder, F.Cu at (183.5, 83.3)
- added R53: 1k, Resistor_SMD:R_0603_1608Metric_Pad1.05x0.95mm_HandSolder, F.Cu at (169.2, 74.4)
- added R54: 1k, Resistor_SMD:R_0603_1608Metric_Pad1.05x0.95mm_HandSolder, F.Cu at (184.5, 125.5)
- added R55: 1k, Resistor_SMD:R_0603_1608Metric_Pad1.05x0.95mm_HandSolder, F.Cu at (168.3, 115.0)
- added R56: 4.7k, Resistor_SMD:R_0603_1608Metric_Pad1.05x0.95mm_HandSolder, F.Cu at (191.5, 59.0)
- added R57: 4.7k, Resistor_SMD:R_0603_1608Metric_Pad1.05x0.95mm_HandSolder, F.Cu at (190.9, 101.7)
- added R58: 4.7k, Resistor_SMD:R_0603_1608Metric_Pad1.05x0.95mm_HandSolder, F.Cu at (92.7, 86.1)
- added R59: 4.7k, Resistor_SMD:R_0603_1608Metric_Pad1.05x0.95mm_HandSolder, F.Cu at (91.1, 86.1)
- added R60: 4.7k, Resistor_SMD:R_0603_1608Metric_Pad1.05x0.95mm_HandSolder, F.Cu at (114.5, 76.7)
- added R61: 4.7k, Resistor_SMD:R_0603_1608Metric_Pad1.05x0.95mm_HandSolder, F.Cu at (116.0, 76.6)
- added R62: 4.7k, Resistor_SMD:R_0603_1608Metric_Pad1.05x0.95mm_HandSolder, F.Cu at (117.3, 90.2)
- added R63: 65Ohm, Resistor_SMD:R_0603_1608Metric_Pad1.05x0.95mm_HandSolder, F.Cu at (81.5, 123.2)
- added REF**: MountingHole_3.2mm_M3, MountingHole:MountingHole_3.2mm_M3, F.Cu at (212.0, 133.5)
- added REF**: MountingHole_3.2mm_M3, MountingHole:MountingHole_3.2mm_M3, F.Cu at (75.0, 133.5)
- added REF**: MountingHole_3.2mm_M3, MountingHole:MountingHole_3.2mm_M3, F.Cu at (212.0, 41.5)
- added REF**: MountingHole_3.2mm_M3, MountingHole:MountingHole_3.2mm_M3, F.Cu at (75.0, 41.5)
- added TP17: TestPoint, Connector_Wire:SolderWirePad_1x01_Drill1.2mm, F.Cu at (108.0, 101.0)
- added U10: TXB0104D, Package_SO:SOIC-14_3.9x8.7mm_P1.27mm, F.Cu at (127.5, 107.5)
- added U11: VNH5019, TurtlebotController:Pololu_VNH5019_Carrier, F.Cu at (181.5, 94.0)
- added U12: VNH5019A-E, Package_SO:ST_MultiPowerSO-30, F.Cu at (148.0, 69.5)
- added U13: VNH5019A-E, Package_SO:ST_MultiPowerSO-30, F.Cu at (147.8, 110.9)
- added U14: VNH5019A-E, Package_SO:ST_MultiPowerSO-30, F.Cu at (179.2, 68.9)
- added U15: VNH5019A-E, Package_SO:ST_MultiPowerSO-30, F.Cu at (179.2, 111.0)
- added U16: ADC128D818, Package_SO:TSSOP-16_4.4x5mm_P0.65mm, F.Cu at (91.6, 92.3)
- added U17: REF3030, Package_TO_SOT_SMD:SOT-23, F.Cu at (95.3, 82.5)
- added U18: MCP23017_SS, Package_SO:SSOP-28_5.3x10.2mm_P0.65mm, F.Cu at (119.1, 83.6)
- added U8: TXB0104D, Package_SO:SOIC-14_3.9x8.7mm_P1.27mm, F.Cu at (127.5, 96.3)
- added U9: VNH5019, TurtlebotController:Pololu_VNH5019_Carrier, F.Cu at (150.0, 94.0)
- J2: value LEFT_MOTOR -> MOTOR_1
- J3: value RIGHT_MOTOR -> MOTOR_2
- R11, R13, R15: value 270Ohm -> 1k
- R12, R14, R16: value 560Ohm -> 1k
- R17: value 270Ohm -> 10k
- R18: value 560Ohm -> 10k
- moved D4 97.7 mm to (201.9, 42.7), turned to 270 degrees
- moved D3 93.8 mm to (198.9, 42.8), turned to 270 degrees
- moved R6 92.5 mm to (201.9, 46.2), turned to 270 degrees
- moved D2 90.0 mm to (195.8, 42.8), turned to 270 degrees
- moved R5 88.4 mm to (198.9, 46.3), turned to 270 degrees
- moved TP4 88.1 mm to (201.9, 49.4), turned to 180 degrees
- moved D1 86.7 mm to (192.8, 42.8), turned to 270 degrees
- moved R4 84.4 mm to (195.8, 46.2), turned to 270 degrees
- moved R3 80.9 mm to (192.8, 46.2), turned to 270 degrees
- moved TP5 79.6 mm to (195.8, 49.4), turned to 180 degrees
- moved TP6 75.6 mm to (192.5, 49.5), turned to 180 degrees
- moved J4 72.6 mm to (171.8, 44.6)
- moved J5 72.6 mm to (178.9, 44.6)
- moved J6 72.6 mm to (185.8, 44.6)
- moved R13 64.1 mm to (143.5, 125.1), turned to 90 degrees
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Connections:
- net LEFT_MOTOR_A renamed MOTOR_1_A
- net LEFT_MOTOR_B renamed MOTOR_1_B
- net RIGHT_MOTOR_A renamed MOTOR_2_A
- net RIGHT_MOTOR_B renamed MOTOR_2_B
- J1 pad 11: Net-(J1-Pad11) -> (no net)
- J1 pad 12: Net-(J1-Pad12) -> (no net)
- J1 pad 13: Net-(J1-Pad13) -> (no net)
- J1 pad 15: Net-(J1-Pad15) -> (no net)
- J1 pad 16: Net-(J1-Pad16) -> (no net)
- J1 pad 18: Net-(J1-Pad18) -> (no net)
- J1 pad 19: TEENSY_MOSI -> (no net)
- J1 pad 21: TEENSY_MISO -> (no net)
- J1 pad 22: Net-(J1-Pad22) -> (no net)
- J1 pad 23: TEENSY_SCK -> (no net)
- J1 pad 24: TEENSY_CS -> (no net)
- J1 pad 26: Net-(J1-Pad26) -> (no net)
- J1 pad 27: Net-(J1-Pad27) -> (no net)
- J1 pad 28: Net-(J1-Pad28) -> (no net)
- J1 pad 29: Net-(J1-Pad29) -> (no net)
- J1 pad 31: Net-(J1-Pad31) -> (no net)
- J1 pad 33: Net-(J1-Pad33) -> (no net)
- J1 pad 35: Net-(J1-Pad35) -> (no net)
- J1 pad 36: Net-(J1-Pad36) -> (no net)
- J1 pad 37: Net-(J1-Pad37) -> (no net)
- J1 pad 38: Net-(J1-Pad38) -> (no net)
- J1 pad 40: Net-(J1-Pad40) -> (no net)
- J1 pad 7: Net-(J1-Pad7) -> (no net)
- J2 pad 4: +5V -> Net-(J2-Pad4)
- J2 pad 5: LEFT_ENCODER_A_5V -> MOTOR_1_ENCODER_A_5V
- J2 pad 6: LEFT_ENCODER_B_5V -> MOTOR_1_ENCODER_B_5V
- J3 pad 4: +5V -> Net-(J3-Pad4)
- J3 pad 5: RIGHT_ENCODER_A_5V -> MOTOR_2_ENCODER_A_5V
- J3 pad 6: RIGHT_ENCODER_B_5V -> MOTOR_2_ENCODER_B_5V
- R11 pad 1: LEFT_ENCODER_A_5V -> MOTOR_1_DIAGA
- R11 pad 2: LEFT_ENCODER_A_3.3V -> Net-(R11-Pad2)
- R12 pad 1: LEFT_ENCODER_A_3.3V -> MOTOR_1_DIAGB
- R12 pad 2: GND -> Net-(R12-Pad2)
- R13 pad 1: LEFT_ENCODER_B_5V -> MOTOR_3_DIAGA
- R13 pad 2: LEFT_ENCODER_B_3.3V -> Net-(R13-Pad2)
- R14 pad 1: LEFT_ENCODER_B_3.3V -> MOTOR_3_DIAGB
- R14 pad 2: GND -> Net-(R14-Pad2)
- R15 pad 1: RIGHT_ENCODER_A_5V -> MOTOR_1_PWM
- R15 pad 2: RIGHT_ENCODER_A_3.3V -> Net-(R15-Pad2)
- R16 pad 1: RIGHT_ENCODER_A_3.3V -> MOTOR_3_PWM
- R16 pad 2: GND -> Net-(R16-Pad2)
- R17 pad 1: RIGHT_ENCODER_B_5V -> Net-(R15-Pad2)
- R17 pad 2: RIGHT_ENCODER_B_3.3V -> GND
- R18 pad 1: RIGHT_ENCODER_B_3.3V -> Net-(R16-Pad2)
- U1 pad 10: TEENSY_TX -> MOTOR_2_PWM
- U1 pad 11: RIGHT_MOTOR_DIAGB -> MOTOR_3_PWM
- U1 pad 12: TEENSY_CS -> MOTOR_4_PWM
- U1 pad 13: TEENSY_MOSI -> MPU_INTERRUPT
- U1 pad 14: TEENSY_MISO -> TEENSY_DEBUG
- U1 pad 15: Net-(U1-Pad15) -> (no net)
- U1 pad 18: Net-(U1-Pad18) -> (no net)
- U1 pad 19: Net-(U1-Pad19) -> (no net)
- U1 pad 2: MPU_INTERRUPT -> MOTOR_1_ENCODER_A
- U1 pad 20: TEENSY_SCK -> TEENSY_HEARTBEAT
- U1 pad 21: LEFT_MOTOR_PWM -> MOTOR_4_CS
- U1 pad 22: RIGHT_MOTOR_PWM -> MOTOR_3_CS
- U1 pad 23: LEFT_MOTOR_CURRENT -> MOTOR_2_CS
- U1 pad 24: RIGHT_MOTOR_CURRENT -> MOTOR_1_CS
- U1 pad 27: LEFT_MOTOR_DIAGA -> TEENSY_TX
- U1 pad 28: LEFT_MOTOR_DIAGB -> TEENSY_RX
- U1 pad 3: TEENSY_HEARTBEAT -> MOTOR_1_ENCODER_B
- U1 pad 34: Net-(U1-Pad34) -> (no net)
- U1 pad 4: RIGHT_ENCODER_A_3.3V -> MOTOR_2_ENCODER_A
- U1 pad 5: RIGHT_ENCODER_B_3.3V -> MOTOR_2_ENCODER_B
- U1 pad 6: LEFT_ENCODER_A_3.3V -> MOTOR_3_ENCODER_A
- U1 pad 7: LEFT_ENCODER_B_3.3V -> MOTOR_3_ENCODER_B
- U1 pad 8: RIGHT_MOTOR_DIAGA -> MOTOR_1_PWM
- U1 pad 9: TEENSY_RX -> MOTOR_4_ENCODER_A
- U2 pad 4: Net-(U2-Pad4) -> (no net)
- U3 pad 1: Net-(U3-Pad1) -> MOTOR_1_INA
- U3 pad 14: Net-(F2-Pad1) -> +12V
- U3 pad 2: LEFT_MOTOR_DIAGA -> MOTOR_1_DIAGA
- U3 pad 3: LEFT_MOTOR_PWM -> MOTOR_1_PWM
- U3 pad 4: LEFT_MOTOR_CURRENT -> MOTOR_1_CS
- U3 pad 5: LEFT_MOTOR_DIAGB -> MOTOR_1_DIAGB
- U3 pad 6: Net-(U3-Pad6) -> MOTOR_1_INB
- U3 pad 9: LEFT_MOTOR_OUT -> (no net)
- U4 pad 1: Net-(U4-Pad1) -> MOTOR_2_INA
- U4 pad 14: Net-(F3-Pad1) -> +12V
- U4 pad 2: RIGHT_MOTOR_DIAGA -> MOTOR_2_DIAGA
- U4 pad 3: RIGHT_MOTOR_PWM -> MOTOR_2_PWM
- U4 pad 4: RIGHT_MOTOR_CURRENT -> MOTOR_2_CS
- U4 pad 5: RIGHT_MOTOR_DIAGB -> MOTOR_2_DIAGB
- U4 pad 6: Net-(U4-Pad6) -> MOTOR_2_INB
- U4 pad 9: RIGHT_MOTOR_OUT -> (no net)
- U6 pad 5: Net-(U6-Pad5) -> (no net)
- U6 pad 6: 5v_PG -> (no net)
- U6 pad 7: Net-(U6-Pad7) -> (no net)
Routing:
- net +3V3: track 212.4 -> 562.8 mm, vias 8 -> 26
- net GND: track 22.2 -> 232.8 mm, vias 36 -> 99
- net +12V: track 278.6 -> 465.6 mm, vias 4 -> 6
- net MOTOR_4_CS: track 0.00 -> 157.8 mm, vias 0 -> 2
- net MOTOR_2_CS: track 0.00 -> 148.6 mm, vias 0 -> 13
- net +5V: track 262.1 -> 400.2 mm, vias 7 -> 27
- net MOTOR_4_PWM: track 0.00 -> 118.0 mm, vias 0 -> 3
- net MOTOR_3_CS: track 0.00 -> 113.5 mm, vias 0 -> 2
- net MOTOR_4_INB: track 0.00 -> 112.5 mm, vias 0 -> 1
- net MOTOR_2_ENCODER_B_5V: track 0.00 -> 112.3 mm, vias 0 -> 3
- net MOTOR_3_A: track 0.00 -> 109.6 mm, vias 0 -> 6
- net MOTOR_1_A: track 11.1 -> 119.4 mm, vias 0 -> 3
- net MOTOR_2_ENCODER_A_5V: track 0.00 -> 104.0 mm, vias 0 -> 4
- net MOTOR_2_PWM: track 0.00 -> 102.2 mm, vias 0 -> 7
- net LEFT_ENCODER_B_3.3V: track 101.4 -> 0.00 mm, vias 8 -> 0
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- added copper zone on F.Cu, net MOTOR_1_A
- added copper zone on F.Cu, net MOTOR_1_B
- added copper zone on F.Cu, net MOTOR_2_A
- added copper zone on F.Cu, net MOTOR_2_B
- added copper zone on F.Cu, net MOTOR_3_A
- added copper zone on F.Cu, net MOTOR_3_B
- added copper zone on F.Cu, net MOTOR_4_A
- added copper zone on F.Cu, net MOTOR_4_B
- added copper zone on F.Cu, net Net-(C16-Pad1)
- added copper zone on F.Cu, net Net-(C18-Pad1)
- added copper zone on F.Cu, net Net-(C24-Pad1)
- added copper zone on F.Cu, net Net-(C26-Pad1)
Other:
- board size 110 x 80 mm -> 147 x 102 mm

Commit message: RevB
Parts:
- removed D1: 12V_OK, LED_SMD:LED_0603_1608Metric_Pad1.05x0.95mm_HandSolder
- removed D6: TEENSY_HEARTBEAT, LED_SMD:LED_0603_1608Metric_Pad1.05x0.95mm_HandSolder
- removed TP15: SDA_0, TestPoint:TestPoint_Pad_D1.5mm
- added 12V: 12V_OK, LED_SMD:LED_0603_1608Metric_Pad1.05x0.95mm_HandSolder, F.Cu at (192.8, 42.8)
- added HEARTBEAT: TEENSY_HEARTBEAT, LED_SMD:LED_0603_1608Metric_Pad1.05x0.95mm_HandSolder, F.Cu at (79.8, 126.8)
- added JP14: Jumper_3_Bridged12, Jumper:SolderJumper-3_P1.3mm_Bridged12_RoundedPad1.0x1.5mm, F.Cu at (132.5, 117.0)
- added SDA: SDA_0, TestPoint:TestPoint_Pad_D1.5mm, F.Cu at (73.5, 66.5)
- turned JP11 to 0 degrees
- renumbered J5 to 3.3V, D4 to 3.3V, J4 to 5V, D2 to 5V, J6 to BAT, D13 to DEBUG, D5 to RPI, JP3 to RPI_VCC, JP2 to SCL, TP16 to SCL, JP1 to SDA, JP6 to VCC, JP7 to VCC, JP8 to VCC, JP9 to VCC
Connections:
- C11 pad 2: +5V -> Net-(C11-Pad2)
- C9 pad 2: +5V -> Net-(C11-Pad2)
- J1 pad 11: (no net) -> Net-(J1-Pad11)
- J1 pad 12: (no net) -> Net-(J1-Pad12)
- J1 pad 13: (no net) -> Net-(J1-Pad13)
- J1 pad 15: (no net) -> Net-(J1-Pad15)
- J1 pad 16: (no net) -> Net-(J1-Pad16)
- J1 pad 18: (no net) -> Net-(J1-Pad18)
- J1 pad 19: (no net) -> TEENSY_MOSI
- J1 pad 21: (no net) -> TEENSY_MISO
- J1 pad 22: (no net) -> Net-(J1-Pad22)
- J1 pad 23: (no net) -> TEENSY_SCK
- J1 pad 24: (no net) -> TEENSY_CS
- J1 pad 26: (no net) -> Net-(J1-Pad26)
- J1 pad 27: (no net) -> Net-(J1-Pad27)
- J1 pad 28: (no net) -> Net-(J1-Pad28)
- J1 pad 29: (no net) -> Net-(J1-Pad29)
- J1 pad 31: (no net) -> Net-(J1-Pad31)
- J1 pad 33: (no net) -> Net-(J1-Pad33)
- J1 pad 35: (no net) -> Net-(J1-Pad35)
- J1 pad 36: (no net) -> Net-(J1-Pad36)
- J1 pad 37: (no net) -> Net-(J1-Pad37)
- J1 pad 38: (no net) -> Net-(J1-Pad38)
- J1 pad 40: (no net) -> Net-(J1-Pad40)
- J1 pad 7: (no net) -> Net-(J1-Pad7)
- JP11 pad 1: GND -> +3V3
- JP11 pad 3: +3V3 -> GND
- U1 pad 15: (no net) -> Net-(U1-Pad15)
- U1 pad 18: (no net) -> Net-(U1-Pad18)
- U1 pad 19: (no net) -> Net-(U1-Pad19)
- U1 pad 34: (no net) -> Net-(U1-Pad34)
- U10 pad 14: +5V -> Net-(C11-Pad2)
- U10 pad 6: (no net) -> Net-(U10-Pad6)
- U10 pad 9: (no net) -> Net-(U10-Pad9)
- U11 pad 9: (no net) -> MOTOR_4_OUT
- U12 pad 14: (no net) -> Net-(U12-Pad14)
- U12 pad 17: (no net) -> Net-(U12-Pad17)
- U12 pad 2: (no net) -> Net-(U12-Pad2)
- U12 pad 22: (no net) -> Net-(U12-Pad22)
- U12 pad 24: (no net) -> Net-(U12-Pad24)
- U12 pad 29: (no net) -> Net-(U12-Pad29)
- U12 pad 6: (no net) -> Net-(U12-Pad6)
- U13 pad 14: (no net) -> Net-(U13-Pad14)
- U13 pad 17: (no net) -> Net-(U13-Pad17)
- U13 pad 2: (no net) -> Net-(U13-Pad2)
- U13 pad 22: (no net) -> Net-(U13-Pad22)
- U13 pad 24: (no net) -> Net-(U13-Pad24)
- U13 pad 29: (no net) -> Net-(U13-Pad29)
- U13 pad 6: (no net) -> Net-(U13-Pad6)
- U14 pad 14: (no net) -> Net-(U14-Pad14)
- U14 pad 17: (no net) -> Net-(U14-Pad17)
- U14 pad 2: (no net) -> Net-(U14-Pad2)
- U14 pad 22: (no net) -> Net-(U14-Pad22)
- U14 pad 24: (no net) -> Net-(U14-Pad24)
- U14 pad 29: (no net) -> Net-(U14-Pad29)
- U14 pad 6: (no net) -> Net-(U14-Pad6)
- U15 pad 14: (no net) -> Net-(U15-Pad14)
- U15 pad 17: (no net) -> Net-(U15-Pad17)
- U15 pad 2: (no net) -> Net-(U15-Pad2)
- U15 pad 22: (no net) -> Net-(U15-Pad22)
- U15 pad 24: (no net) -> Net-(U15-Pad24)
- U15 pad 29: (no net) -> Net-(U15-Pad29)
- U15 pad 6: (no net) -> Net-(U15-Pad6)
- U16 pad 10: (no net) -> Net-(U16-Pad10)
- U16 pad 6: (no net) -> Net-(U16-Pad6)
- U16 pad 7: (no net) -> Net-(U16-Pad7)
- U16 pad 8: (no net) -> Net-(U16-Pad8)
- U16 pad 9: (no net) -> Net-(U16-Pad9)
- U18 pad 11: (no net) -> Net-(U18-Pad11)
- U18 pad 14: (no net) -> Net-(U18-Pad14)
- U18 pad 19: (no net) -> Net-(U18-Pad19)
- U18 pad 20: (no net) -> Net-(U18-Pad20)
- U2 pad 4: (no net) -> Net-(U2-Pad4)
- U3 pad 9: (no net) -> MOTOR_1_OUT
- U4 pad 9: (no net) -> MOTOR_2_OUT
- U6 pad 5: (no net) -> Net-(U6-Pad5)
- U6 pad 6: (no net) -> 5v_PG
- U6 pad 7: (no net) -> Net-(U6-Pad7)
- U8 pad 14: +5V -> Net-(C11-Pad2)
- U8 pad 6: (no net) -> Net-(U8-Pad6)
- U8 pad 9: (no net) -> Net-(U8-Pad9)
- U9 pad 9: (no net) -> MOTOR_3_OUT
Routing:
- net Net-(C11-Pad2): track 0.00 -> 39.4 mm, vias 0 -> 3
- net +3V3: track 562.8 -> 570.9 mm, vias 26 -> 27
- net +5V: track 400.2 -> 404.8 mm, vias 27 -> 29
- net MOTOR_2_ENCODER_A_5V: track 104.0 -> 105.3 mm
- net TEENSY_HEARTBEAT: track 28.7 -> 27.9 mm
- net GND: track 232.8 -> 233.4 mm
Other:
- board text added: "- 3.3V"
- board text added: "- 5V"
- board text added: "- BAT"
- board text added: "5V"
- board text added: "A"
- board text added: "Abiel Fernández TurtlebotController Rev. B 2020"
- board text added: "B"
- board text added: "MOTOR 1"
- board text added: "MOTOR 2"
- board text added: "MOTOR 3"
- board text added: "MOTOR 4"
- board text removed: "- +"
- board text removed: "Abiel Fernández TurtlebotController Rev. A 2019"

Commit message: Rev B
Parts:
- added REF**: Symbol_HighVoltage_Type1_CopperTop_Big, Symbol:Symbol_HighVoltage_Type1_CopperTop_Big, F.Cu at (116.8, 50.8)

Commit message: Added readme (#1)
* Add media

* Create README.md
Other:
- net class Default removed
- net class Power removed
